Commit message: Update urdf and rviz file

File: daVinciCore/urdf/daVinci_jhu.urdf (robot description, URDF)
Before this commit: robot daVinci, 10 links, 9 joints
Links:
- removed link mounting_base_link
- removed link mounting_platform
- removed link outer_pitch_base_link
- removed link tool_adaptor_link
- removed link tool_link
- added link outer_pitch_back_link; visual mesh filename=package://daVinciCore/meshes/outer_pitch_back.dae
- added link psm_base_link; visual mesh filename=package://daVinciCore/meshes/psm_base.dae
- added link tool_main_link; visual mesh filename=package://daVinciCore/meshes/tool_main.dae
- added link tool_wrist_link; visual mesh filename=package://daVinciCore/meshes/tool_wrist_link.dae
- added link tool_wrist_sca_ee_link_1; visual mesh filename=package://daVinciCore/meshes/tool_wrist_sca_link_2.dae
- added link tool_wrist_sca_ee_link_2; visual mesh filename=package://daVinciCore/meshes/tool_wrist_sca_link_2.dae
- added link tool_wrist_sca_link; visual mesh filename=package://daVinciCore/meshes/tool_wrist_sca_link.dae
- added link tool_wrist_sca_shaft_link; visual mesh filename=package://daVinciCore/meshes/tool_wrist_sca_shaft_link.dae
- added link tool_wrist_shaft_link; visual mesh filename=package://daVinciCore/meshes/tool_wrist_shaft_link.dae
- link outer_insertion_link: mass 0.01 -> None; geometry visual mesh filename=package://daVinciCore/meshes/outer_insertion.dae
- link outer_pitch_bottom_link: mass 0.01 -> None; geometry visual mesh filename=package://daVinciCore/meshes/outer_pitch_bottom.dae
- link outer_pitch_front_link: mass 0.01 -> None; geometry visual mesh filename=package://daVinciCore/meshes/outer_pitch_front.dae
- link outer_pitch_top_link: mass 0.01 -> None; geometry visual mesh filename=package://daVinciCore/meshes/outer_pitch_top.dae
- link outer_yaw_link: mass 0.01 -> None; geometry visual mesh filename=package://daVinciCore/meshes/outer_yaw.dae
Joints:
- removed joint mounting_base_joint
- removed joint outer_pitch_base_joint
- removed joint outer_pitch_bottom_joint
- removed joint outer_pitch_front_joint
- removed joint outer_pitch_top_joint
- removed joint tool_insertion_joint
- removed joint tool_joint
- added joint outer_pitch_joint_1: type revolute, parent outer_yaw_link, child outer_pitch_back_link, origin xyz=0 0.0295 0.1495 rpy=-1.5708 -1.5708 0, axis 0 0 1, limit lower=-0.7854 upper=0.7854 effort=1000 velocity=.4
- added joint outer_pitch_joint_2: type continuous, parent outer_yaw_link, child outer_pitch_front_link, origin xyz=0 0.0295 0.0595 rpy=-1.5708 -1.5708 0, axis 0 0 1, mimic joint=outer_pitch_joint_1 multiplier=1
- added joint outer_pitch_joint_3: type continuous, parent outer_pitch_back_link, child outer_pitch_bottom_link, origin xyz=0.04178 0.15007 -0.0137 rpy=0 0 0, axis 0 0 1, mimic joint=outer_pitch_joint_1 multiplier=-1
- added joint outer_pitch_joint_4: type continuous, parent outer_pitch_back_link, child outer_pitch_top_link, origin xyz=0.04209 0.18695 -0.02412 rpy=0 0 0, axis 0 0 1, mimic joint=outer_pitch_joint_1 multiplier=-1
- added joint outer_pitch_joint_5: type continuous, parent outer_pitch_bottom_link, child outer_insertion_link, origin xyz=-0.520 0 -0.0175 rpy=0 0 0, axis 0 0 1, mimic joint=outer_pitch_joint_1 multiplier=1
- added joint outer_roll_joint: type revolute, parent tool_main_link, child tool_wrist_link, origin xyz=0 0 0.36680 rpy=0 0 0, axis 0 0 1, limit lower=-2.2689 upper=2.2689 effort=1000 velocity=.4
- added joint outer_roll_shaft_joint: type fixed, parent tool_wrist_link, child tool_wrist_shaft_link, origin xyz=0 0 0.0091 rpy=0 0 0, axis 0 0 1
- added joint outer_wrist_open_angle_joint_1: type revolute, parent tool_wrist_sca_shaft_link, child tool_wrist_sca_ee_link_1, origin xyz=0 0 0 rpy=0 0 0, axis 0 0 1, limit lower=0 upper=1.5707 effort=1000 velocity=.4
- added joint outer_wrist_open_angle_joint_2: type revolute, parent tool_wrist_sca_shaft_link, child tool_wrist_sca_ee_link_2, origin xyz=0 0 0 rpy=0 0 0, axis 0 0 1, limit lower=-1.5707 upper=1.5707 effort=1000 velocity=.4, mimic joint=outer_wrist_open_angle_joint_1 multiplier=-1
- added joint outer_wrist_pitch_joint: type revolute, parent tool_wrist_shaft_link, child tool_wrist_sca_link, origin xyz=0 0 0 rpy=-1.5708 -1.5708 0, axis 0 0 1, limit lower=-1.5707 upper=1.5707 effort=1000 velocity=.4
- added joint outer_wrist_yaw_joint: type revolute, parent tool_wrist_sca_link, child tool_wrist_sca_shaft_link, origin xyz=0.0089 0 0 rpy=-1.5708 -1.5708 0, axis 0 0 1, limit lower=-1.3963 upper=1.3963 effort=1000 velocity=.4
- joint outer_insertion_joint: axis 0 1 0 -> 0 0 1; child outer_insertion_link -> tool_main_link; limit lower=-0.7854 upper=0.7854 effort=1000 velocity=.4 -> lower=0 upper=0.240 effort=1000 velocity=.4; origin xyz=0.510 0.003 0 rpy=0 0 0 -> xyz=-0.0403 0.23622 0 rpy=1.5708 0 0; parent outer_pitch_bottom_link -> outer_insertion_link; type revolute -> prismatic
- joint outer_yaw_joint: axis 1 0 0 -> 0 0 1; origin xyz=0.094 0.0525 0.147 rpy=0 0 0 -> xyz=0.0 0.0 0.0 rpy=1.5708 -1.5708 0; parent mounting_base_link -> psm_base_link
