Commit message: updated file

File: MTM_CAD_Model/meshes/MTM_model.urdf (robot description, URDF)
Before this commit: robot DaVinci Robot, 11 links, 10 joints
Joints:
- joint ABottom_to_WristPlat: limit lower=1.57 upper=1.57 effort=100.0 velocity=1000 -> lower=0 upper=3.14159 effort=100.0 velocity=1000; origin xyz=-.3148 -.02746 0 rpy=3.14 1.57 1.57 -> xyz=-.3148 -.02646 0 rpy=3.14 1.57 1.57
- joint AparX2_to_link: limit lower=-3.14159 upper=3.14159 effort=100.0 velocity=1000 -> lower=0 upper=0 effort=100.0 velocity=1000
- joint Aparallel_to_Abottom: limit lower=1.57 upper=1.57 effort=100.0 velocity=1000 -> lower=.33 upper=2.35 effort=100.0 velocity=1000
- joint OutPitchSh_to_APar_X2: limit lower=-3.14159 upper=3.14159 effort=100.0 velocity=1000 -> lower=-1.14 upper=1.0 effort=100.0 velocity=1000
- joint OutPitchSh_to_AParallel: limit lower=0 upper=3.14159 effort=100.0 velocity=1000 -> lower=-1.14 upper=1.0 effort=100.0 velocity=1000
- joint Pitch_to_yaw: limit lower=-3.14159 upper=3.14159 effort=100.0 velocity=1000 -> lower=-2.60 upper=2.50 effort=100.0 velocity=1000
- joint Top_panel_to_OutPitchSh: limit lower=0.0 upper=3.14159 effort=1000.0 velocity=1000 -> lower=-.70 upper=2.16 effort=1000.0 velocity=1000
- joint WristPlat_to_WristPitch: limit lower=0.0 upper=3.14159 effort=100.0 velocity=1000 -> lower=-1.57 upper=3.14159 effort=100.0 velocity=1000
- joint Yaw_to_Roll: limit lower=-2.57 upper=2.57 effort=100.0 velocity=1000 -> lower=-3.14159 upper=3.14159 effort=100.0 velocity=1000

Commit message: updated file with point mass

File: MTM_CAD_Model/meshes/MTM_model.urdf (robot description, URDF)
Before this commit: robot DaVinci Robot, 11 links, 10 joints
Links:
- link A_Bottom: mass None -> 800
- link A_Par_x2: mass None -> 500
- link A_Parallel: mass None -> 900
- link Link_APar: mass 10 -> 300
- link OutPitch_S: mass None -> 1000
- link Top_Panel: mass None -> 900
- link Wrist_Pitch: mass None -> 250
- link Wrist_Platform: mass None -> 300
- link Wrist_Roll: mass None -> 140
- link Wrist_Yaw: mass None -> 200
- link base_link: geometry 
