Commit message: renamed dv_model to irk_model

File: irk_model/urdf/daVinci_jhu.urdf (robot description, URDF)
Before this commit: robot daVinci, 14 links, 13 joints
Links:
- link outer_insertion_link: geometry visual mesh filename=package://irk_model/meshes/outer_insertion.dae
- link outer_pitch_back_link: geometry visual mesh filename=package://irk_model/meshes/outer_pitch_back.dae
- link outer_pitch_bottom_link: geometry visual mesh filename=package://irk_model/meshes/outer_pitch_bottom.dae
- link outer_pitch_front_link: geometry visual mesh filename=package://irk_model/meshes/outer_pitch_front.dae
- link outer_pitch_top_link: geometry visual mesh filename=package://irk_model/meshes/outer_pitch_top.dae
- link outer_yaw_link: geometry visual mesh filename=package://irk_model/meshes/outer_yaw.dae
- link psm_base_link: geometry visual mesh filename=package://irk_model/meshes/psm_base.dae
- link tool_main_link: geometry visual mesh filename=package://irk_model/meshes/tool_main.dae
- link tool_wrist_link: geometry visual mesh filename=package://irk_model/meshes/tool_wrist_link.dae
- link tool_wrist_sca_ee_link_1: geometry visual mesh filename=package://irk_model/meshes/tool_wrist_sca_link_2.dae
- link tool_wrist_sca_ee_link_2: geometry visual mesh filename=package://irk_model/meshes/tool_wrist_sca_link_2.dae
- link tool_wrist_sca_link: geometry visual mesh filename=package://irk_model/meshes/tool_wrist_sca_link.dae
- link tool_wrist_sca_shaft_link: geometry visual mesh filename=package://irk_model/meshes/tool_wrist_sca_shaft_link.dae
- link tool_wrist_shaft_link: geometry visual mesh filename=package://irk_model/meshes/tool_wrist_shaft_link.dae
