Commit message: added psm_jhu.urdf.xacro and updated related files

File: irk_model/model/mtm.urdf.xacro (robot description, xacro)
@@ -112,20 +112,20 @@
       </inertial>
     </link>
-    <link name="${prefix}front_parallel_link">
-      <visual>
-        <geometry>
-          <mesh filename="package://irk_model/meshes/mtm/Link.dae"/>
-        </geometry>
-      </visual>
-      <collision>
-        <geometry>
-          <mesh filename="package://irk_model/meshes/mtm/Link.STL"/>
-        </geometry>
-      </collision>
-      <inertial>
-        <mass value="0.8"/>
-        <inertia ixx="8.0" ixy="0.0" ixz="0.0" iyy="8.0" iyz="0.0" izz="8.0"/>
-      </inertial>
-    </link>
+    <!-- <link name="${prefix}front_parallel_link"> -->
+    <!--   <visual> -->
+    <!--     <geometry> -->
+    <!--       <mesh filename="package://irk_model/meshes/mtm/Link.dae"/> -->
+    <!--     </geometry> -->
+    <!--   </visual> -->
+    <!--   <collision> -->
+    <!--     <geometry> -->
+    <!--       <mesh filename="package://irk_model/meshes/mtm/Link.STL"/> -->
+    <!--     </geometry> -->
+    <!--   </collision> -->
+    <!--   <inertial> -->
+    <!--     <mass value="0.8"/> -->
+    <!--     <inertia ixx="8.0" ixy="0.0" ixz="0.0" iyy="8.0" iyz="0.0" izz="8.0"/> -->
+    <!--   </inertial>  -->
+    <!-- </link> -->
     <joint name="${prefix}shoulder_pitch_joint" type="revolute">
       <parent link="${prefix}outer_yaw_link"/>
@@ -147,15 +147,14 @@
       <limit effort="100.0" lower="${-PI/2}" upper="${PI/2}" velocity="10"/>
       <joint_properties damping="1.0" friction="0.0"/>
-    </joint>
-    <joint name="${prefix}elbow_pitch_parallel_joint" type="revolute">
-      <parent link="${prefix}top_parallel_link"/>
-      <child link="${prefix}front_parallel_link"/>
-      <origin rpy="0 0 0" xyz=".1011 0 -0.03"/>
-      <axis xyz="0 0 1"/>
-      <!--limit effort and velocity picked arbitrarily check-->
-      <!-- front_parallel_link will not move from its attached link (A_Parx2)-->
-      <limit effort="100.0" lower="${-PI/4}" upper="${PI/4}" velocity="10"/>
-      <joint_properties damping="1.0" friction="0.0"/>
-    </joint>
+      <mimic joint="${prefix}shoulder_pitch_joint" multiplier="1"/>
+    </joint>
+    <!-- <joint name="${prefix}elbow_pitch_parallel_joint" type="revolute"> -->
+    <!--   <parent link="${prefix}top_parallel_link"/> -->
+    <!--   <child link="${prefix}front_parallel_link"/> -->
+    <!--   <origin rpy="0 0 0" xyz=".1011 0 -0.03"/> -->
+    <!--   <axis xyz="0 0 1"/> -->
+    <!--   <limit effort="100.0" lower="${-PI/4}" upper="${PI/4}" velocity="10"/> -->
+    <!--   <joint_properties damping="1.0" friction="0.0"/> -->
+    <!-- </joint> -->
     <joint name="${prefix}elbow_pitch_joint" type="revolute">
       <parent link="${prefix}back_parallel_link"/>

File: irk_model/model/mtm_right.urdf.xacro (robot description, xacro)
@@ -4,6 +4,7 @@
   <xacro:include filename="$(find irk_model)/model/mtm.urdf.xacro"/>
   <link name="world"/>
-  <xacro:right_mtm
-      prefix=""
-      parent_link="world"/>
+  <xacro:mtm
+      prefix="right_"
+      parent_link="world"
+      xyz="0.25 0.0 1.0" rpy="0.0 0.0 0.0"/>
 </robot>

File: irk_model/model/psm_jhu.urdf (robot description, URDF)
Before this commit: robot irk_psm, 14 links, 13 joints
Links:
- added link world
Joints:
- added joint fixed_joint: type fixed, parent world, child psm_base_link, origin xyz=0.0 0.0 0.0 rpy=0.0 0.0 0.0

Commit message: flipped mtm wrist roll direction + add pi/2 offset to match ISI manual

File: irk_model/model/mtm.urdf.xacro (robot description, xacro)
@@ -272,6 +272,6 @@
       <parent link="${prefix}wrist_yaw_link"/>
       <child link="${prefix}wrist_roll_link"/>  <!-- -.039 & .055 defined from CAD file-->
-      <origin rpy="${-PI/2} 0 0" xyz="0 -.039 0"/>
-      <axis xyz="0 0 1"/>
+      <origin rpy="${-PI/2} ${PI/2} 0" xyz="0 -.039 0"/>
+      <axis xyz="0 0 -1"/>
       <!--rotates about y axis-->
       <!--limit effort and velocity picked arbitrarily check-->
