Commit message: Updated to comply with the files we had before in /rosdavinci

File: dvrk_model/model/mtm_left.urdf.xacro (robot description, xacro)
@@ -5,6 +5,6 @@
   <link name="world"/>
   <xacro:mtm
-      prefix="right_"
+      prefix="left_"
       parent_link="world"
-      xyz="0.25 0.0 1.0" rpy="0.0 0.0 0.0"/>
+      xyz="-0.25 0.0 1.0" rpy="0.0 0.0 0.0"/>
 </robot>

File: dvrk_model/model/psm.urdf.xacro (robot description, xacro)
@@ -3,11 +3,23 @@
   <xacro:macro name="psm" params="prefix parent_link xyz rpy">
     <!-- fixed joint -->
-    <joint name="fixed_joint" type="fixed">
+    <joint name="${prefix}fixed_joint" type="fixed">
       <parent link="${parent_link}"/>
-      <child link="psm_base_link"/>
+      <child link="${prefix}remote_center_link"/>
       <origin rpy="${rpy}" xyz="${xyz}"/>
     </joint>
+    <!-- link rc: remote centre link -->
+    <link name="${prefix}remote_center_link">
+      <visual>
+        <origin rpy="0 0 0" xyz="0 0 0"/>
+      </visual>
+    </link>
+    <!-- fixed joint -->
+    <joint name="${prefix}rc_fixed_joint" type="fixed">
+      <parent link="${prefix}remote_center_link"/>
+      <child link="${prefix}psm_base_link"/>
+      <origin rpy="0 0 0" xyz="0 -0.369 0"/>
+    </joint>
     <!-- link 0: psm base link -->
-    <link name="psm_base_link">
+    <link name="${prefix}psm_base_link">
       <visual>
         <origin rpy="1.5708 0 3.1416" xyz="0.039 -0.03888 -0.07879"/>
@@ -18,7 +30,7 @@
     </link>
     <!-- joint 1 -->
-    <joint name="outer_yaw_joint" type="revolute">
-      <parent link="psm_base_link"/>
-      <child link="outer_yaw_link"/>
+    <joint name="${prefix}outer_yaw_joint" type="revolute">
+      <parent link="${prefix}psm_base_link"/>
+      <child link="${prefix}outer_yaw_link"/>
       <axis xyz="0 0 1"/>
       <origin rpy="1.5708 -1.5708 0" xyz="0.0 0.0 0.0"/>
@@ -26,5 +38,5 @@
     </joint>
     <!-- link 1: outer_yaw -->
-    <link name="outer_yaw_link">
+    <link name="${prefix}outer_yaw_link">
       <visual>
         <!-- <origin rpy="0 0 -1.5708" xyz="0.0125 0 0.1575"/> -->
@@ -36,7 +48,7 @@
     </link>
     <!-- joint 2-1: outer_pitch_1 -->
-    <joint name="outer_pitch_joint_1" type="revolute">
-      <parent link="outer_yaw_link"/>
-      <child link="outer_pitch_back_link"/>
+    <joint name="${prefix}outer_pitch_joint_1" type="revolute">
+      <parent link="${prefix}outer_yaw_link"/>
+      <child link="${prefix}outer_pitch_back_link"/>
       <axis xyz="0 0 1"/>
       <origin rpy="-1.5708 -1.5708 0" xyz="0 0.0295 0.1495"/>
@@ -44,5 +56,5 @@
     </joint>
     <!-- link 2: outer_pitch_back -->
-    <link name="outer_pitch_back_link">
+    <link name="${prefix}outer_pitch_back_link">
       <visual>
         <origin rpy="0 0 -0.27129" xyz="0 0 0"/>
@@ -53,13 +65,13 @@
     </link>
     <!-- joint 2-2: outer_pitch_2 -->
-    <joint name="outer_pitch_joint_2" type="continuous">
-      <parent link="outer_yaw_link"/>
-      <child link="outer_pitch_front_link"/>
+    <joint name="${prefix}outer_pitch_joint_2" type="continuous">
+      <parent link="${prefix}outer_yaw_link"/>
+      <child link="${prefix}outer_pitch_front_link"/>
       <axis xyz="0 0 1"/>
       <origin rpy="-1.5708 -1.5708 0" xyz="0 0.0295 0.0595"/>
-      <mimic joint="outer_pitch_joint_1" multiplier="1"/>
+      <mimic joint="${prefix}outer_pitch_joint_1" multiplier="1"/>
     </joint>
     <!-- link 2-2: outer_pitch_front -->
-    <link name="outer_pitch_front_link">
+    <link name="${prefix}outer_pitch_front_link">
       <visual>
         <origin rpy="0 0 -0.27129" xyz="0 0 0"/>
@@ -71,13 +83,13 @@
     </link>
     <!-- joint 2-3: outer_pitch_3 -->
-    <joint name="outer_pitch_joint_3" type="continuous">
-      <parent link="outer_pitch_back_link"/>
-      <child link="outer_pitch_bottom_link"/>
+    <joint name="${prefix}outer_pitch_joint_3" type="continuous">
+      <parent link="${prefix}outer_pitch_back_link"/>
+      <child link="${prefix}outer_pitch_bottom_link"/>
       <axis xyz="0 0 1"/>
       <origin rpy="0 0 0" xyz="0.04178 0.15007 -0.0137"/>
-      <mimic joint="outer_pitch_joint_1" multiplier="-1"/>
+      <mimic joint="${prefix}outer_pitch_joint_1" multiplier="-1"/>
     </joint>
     <!-- link 2-3: outer_pitch_bottom -->
-    <link name="outer_pitch_bottom_link">
+    <link name="${prefix}outer_pitch_bottom_link">
       <visual>
         <origin rpy="0 -1.5708 0" xyz="0.009 0 0"/>
@@ -88,13 +100,13 @@
     </link>
     <!-- joint 2-4: outer_pitch_4 -->
-    <joint name="outer_pitch_joint_4" type="continuous">
-      <parent link="outer_pitch_back_link"/>
-      <child link="outer_pitch_top_link"/>
+    <joint name="${prefix}outer_pitch_joint_4" type="continuous">
+      <parent link="${prefix}outer_pitch_back_link"/>
+      <child link="${prefix}outer_pitch_top_link"/>
       <axis xyz="0 0 1"/>
       <origin rpy="0 0 0" xyz="0.04209 0.18695 -0.02412"/>
-      <mimic joint="outer_pitch_joint_1" multiplier="-1"/>
+      <mimic joint="${prefix}outer_pitch_joint_1" multiplier="-1"/>
     </joint>
     <!-- link 2-4: outer_pitch_top -->
-    <link name="outer_pitch_top_link">
+    <link name="${prefix}outer_pitch_top_link">
       <visual>
         <origin rpy="0 -1.5708 0" xyz="0.009 0 0"/>
@@ -105,13 +117,13 @@
     </link>
     <!-- joint 2-5: outer_pitch_5 -->
-    <joint name="outer_pitch_joint_5" type="continuous">
-      <parent link="outer_pitch_bottom_link"/>
-      <child link="outer_insertion_link"/>
-      <axis xyz="0 0 1"/>
-      <origin rpy="0 0 0" xyz="-0.520 0 -0.0175"/>
-      <mimic joint="outer_pitch_joint_1" multiplier="1"/>
+    <joint name="${prefix}outer_pitch_joint_5" type="continuous">
+      <parent link="${prefix}outer_pitch_bottom_link"/>
+      <child link="${prefix}outer_insertion_link"/>
+      <axis xyz="0 0 1"/>
+      <origin rpy="0 0 0" xyz="-0.520 0 -0.0155"/>
+      <mimic joint="${prefix}outer_pitch_joint_1" multiplier="1"/>
     </joint>
     <!-- link 2-5: outer_insertion -->
-    <link name="outer_insertion_link">
+    <link name="${prefix}outer_insertion_link">
       <visual>
         <origin rpy="0 -1.5708 1.5708" xyz="0.02528 0.429 0"/>
@@ -122,7 +134,7 @@
     </link>
     <!-- joint 3: insertion -->
-    <joint name="outer_insertion_joint" type="prismatic">
-      <parent link="outer_insertion_link"/>
-      <child link="tool_main_link"/>
+    <joint name="${prefix}outer_insertion_joint" type="prismatic">
+      <parent link="${prefix}outer_insertion_link"/>
+      <child link="${prefix}tool_main_link"/>
       <axis xyz="0 0 1"/>
       <origin rpy="1.5708 0 0" xyz="-0.0403 0.23622 0"/>
@@ -130,5 +142,5 @@
     </joint>
     <!-- link 3: tool_main_link -->
-    <link name="tool_main_link">
+    <link name="${prefix}tool_main_link">
       <visual>
         <origin rpy="0 0 1.5708" xyz="0 0 0"/>
@@ -139,7 +151,7 @@
     </link>
     <!-- joint 4-1: Outer Roll -->
-    <joint name="outer_roll_joint" type="revolute">
-      <parent link="tool_main_link"/>
-      <child link="tool_wrist_link"/>
+    <joint name="${prefix}outer_roll_joint" type="revolute">
+      <parent link="${prefix}tool_main_link"/>
+      <child link="${prefix}tool_wrist_link"/>
       <axis xyz="0 0 1"/>
       <origin rpy="0 0 0" xyz="0 0 0.36680"/>
@@ -147,5 +159,5 @@
     </joint>
     <!-- link 4-1: tool_main_link -->
-    <link name="tool_wrist_link">
+    <link name="${prefix}tool_wrist_link">
       <visual>
         <origin rpy="0 0 1.5708" xyz="0 0 0"/>
@@ -156,12 +168,12 @@
     </link>
     <!-- joint 4-1: Outer Roll shaft -->
-    <joint name="outer_roll_shaft_joint" type="fixed">
-      <parent link="tool_wrist_link"/>
-      <child link="tool_wrist_shaft_link"/>
+    <joint name="${prefix}outer_roll_shaft_joint" type="fixed">
+      <parent link="${prefix}tool_wrist_link"/>
+      <child link="${prefix}tool_wrist_shaft_link"/>
       <axis xyz="0 0 1"/>
       <origin rpy="0 0 0" xyz="0 0 0.0091"/>
     </joint>
     <!-- link 4-1: tool_wrist_shaft_link -->
-    <link name="tool_wrist_shaft_link">
+    <link name="${prefix}tool_wrist_shaft_link">
       <visual>
         <origin rpy="1.5708 0 0" xyz="0 0.00401 0"/>
@@ -172,7 +184,7 @@
     </link>
     <!-- joint 5: Outer wrist pitch joint -->
-    <joint name="outer_wrist_pitch_joint" type="revolute">
-      <parent link="tool_wrist_shaft_link"/>
-      <child link="tool_wrist_sca_link"/>
+    <joint name="${prefix}outer_wrist_pitch_joint" type="revolute">
+      <parent link="${prefix}tool_wrist_shaft_link"/>
+      <child link="${prefix}tool_wrist_sca_link"/>
       <axis xyz="0 0 1"/>
       <origin rpy="-1.5708 -1.5708 0" xyz="0 0 0"/>
@@ -180,5 +192,5 @@
     </joint>
     <!-- link 5: tool_wrist_sca_link -->
-    <link name="tool_wrist_sca_link">
+    <link name="${prefix}tool_wrist_sca_link">
       <visual>
         <!-- <origin rpy="0 3.1416 0" xyz="0 0 0"/> -->
@@ -190,7 +202,7 @@
     </link>
     <!-- joint 5-2: Outer wristyaw joint -->
-    <joint name="outer_wrist_yaw_joint" type="revolute">
-      <parent link="tool_wrist_sca_link"/>
-      <child link="tool_wrist_sca_shaft_link"/>
+    <joint name="${prefix}outer_wrist_yaw_joint" type="revolute">
+      <parent link="${prefix}tool_wrist_sca_link"/>
+      <child link="${prefix}tool_wrist_sca_shaft_link"/>
       <axis xyz="0 0 1"/>
       <origin rpy="-1.5708 -1.5708 0" xyz="0.0089 0 0"/>
@@ -199,5 +211,5 @@
     </joint>
     <!-- link 5-2: tool_wrist_sca_shaft_link -->
-    <link name="tool_wrist_sca_shaft_link">
+    <link name="${prefix}tool_wrist_sca_shaft_link">
       <visual>
         <origin rpy="0 0 0" xyz="0 0 -0.0025"/>
@@ -208,7 +220,7 @@
     </link>
     <!-- joint 6-1: Outer open angle 1  -->
-    <joint name="outer_wrist_open_angle_joint_1" type="revolute">
-      <parent link="tool_wrist_sca_shaft_link"/>
-      <child link="tool_wrist_sca_ee_link_1"/>
+    <joint name="${prefix}outer_wrist_open_angle_joint_1" type="revolute">
+      <parent link="${prefix}tool_wrist_sca_shaft_link"/>
+      <child link="${prefix}tool_wrist_sca_ee_link_1"/>
       <axis xyz="0 0 1"/>
       <origin rpy="0 0 0" xyz="0 0 0"/>
@@ -217,5 +229,5 @@
     </joint>
     <!-- link 6-1: Outer open angle link 1 -->
-    <link name="tool_wrist_sca_ee_link_1">
+    <link name="${prefix}tool_wrist_sca_ee_link_1">
       <visual>
         <origin rpy="0 0 0" xyz="0 0 0"/>
@@ -226,14 +238,14 @@
     </link>
     <!-- joint 6-2: Outer open angle 2   -->
-    <joint name="outer_wrist_open_angle_joint_2" type="revolute">
-      <parent link="tool_wrist_sca_shaft_link"/>
-      <child link="tool_wrist_sca_ee_link_2"/>
+    <joint name="${prefix}outer_wrist_open_angle_joint_2" type="revolute">
+      <parent link="${prefix}tool_wrist_sca_shaft_link"/>
+      <child link="${prefix}tool_wrist_sca_ee_link_2"/>
       <axis xyz="0 0 1"/>
       <origin rpy="0 0 0" xyz="0 0 0"/>
       <limit lower="-1.5707" upper="1.5707" velocity=".4" effort="1000"/>
-      <mimic joint="outer_wrist_open_angle_joint_1" multiplier="-1"/>
+      <mimic joint="${prefix}outer_wrist_open_angle_joint_1" multiplier="-1"/>
     </joint>
     <!-- link 6-2: Outer open angle link 2 -->
-    <link name="tool_wrist_sca_ee_link_2">
+    <link name="${prefix}tool_wrist_sca_ee_link_2">
       <visual>
         <origin rpy="0 3.1516 0" xyz="0 0 0"/>

File: dvrk_model/model/psm_two.urdf.xacro (robot description, xacro)
@@ -5,6 +5,6 @@
   <link name="world"/>
   <xacro:psm
-      prefix="one_"
+      prefix="two_"
       parent_link="world"
-      xyz="-0.25 0.0 0.5" rpy="0.0 0.0 3.1415926"/>
+      xyz="0.25 0.0 0.5" rpy="0.0 0.0 -3.1415926"/>
 </robot>
