Commit message: Changed tabs to spaces

File: dvrk_model/model/both_psms.urdf.xacro (robot description, xacro)
@@ -4,19 +4,19 @@
   <xacro:include filename="$(find dvrk_model)/model/psm.urdf.xacro"/>
   <link name="world">
-						<origin xyz="0.0 0.0 0.0"/>
-		</link>
-		<joint name="world_joint" type="fixed">
-						<parent link="world"/>
-						<child link="camera"/>
-						<origin rpy="0.0 0.0 0.0" xyz="0.0 0.0 0.0"/>
-		</joint>
-		<link name="camera">
-		<origin rpy="0.0 0.0 0.0" xyz="0.0 0.2 0.8"/>
-		</link>
+      <origin xyz="0.0 0.0 0.0"/>
+  </link>
+  <joint name="world_joint" type="fixed">
+      <parent link="world"/>
+      <child link="camera"/>
+      <origin rpy="0.0 0.0 0.0" xyz="0.0 0.0 0.0"/>
+  </joint>
+  <link name="camera">
+  <origin rpy="0.0 0.0 0.0" xyz="0.0 0.2 0.8"/>
+  </link>
   <xacro:psm
       prefix="one_"
       parent_link="camera"
       xyz="-0.25 0.0 0.5" rpy="0.0 0.0 3.1415926"/>
-		<xacro:psm
+  <xacro:psm
       prefix="two_"
       parent_link="camera"
