Commit message: renamed irk_model to dvrk_model

File: dvrk_model/model/mtm.urdf.xacro (robot description, xacro)
@@ -2,5 +2,5 @@
 <robot name="mtm" xmlns:xacro="http://www.ros.org/wiki/xacro">
   <!-- Colors -->
-  <xacro:include filename="$(find irk_model)/model/common.urdf.xacro"/>
+  <xacro:include filename="$(find dvrk_model)/model/common.urdf.xacro"/>
   <!-- Macro for the da Vinci Master Console -->
   <xacro:macro name="master_console" params="prefix parent_link xyz rpy">
@@ -38,10 +38,10 @@
       <visual>
         <geometry>
-          <mesh filename="package://irk_model/meshes/mtm/Top Panel.dae"/>
-        </geometry>
-      </visual>
-      <collision>
-        <geometry>
-          <mesh filename="package://irk_model/meshes/mtm/Top Panel.STL"/>
+          <mesh filename="package://dvrk_model/meshes/mtm/Top Panel.dae"/>
+        </geometry>
+      </visual>
+      <collision>
+        <geometry>
+          <mesh filename="package://dvrk_model/meshes/mtm/Top Panel.STL"/>
         </geometry>
       </collision>
@@ -67,10 +67,10 @@
       <visual>
         <geometry>
-          <mesh filename="package://irk_model/meshes/mtm/OutPitch_Shoulder.dae"/>
-        </geometry>
-      </visual>
-      <collision>
-        <geometry>
-          <mesh filename="package://irk_model/meshes/mtm/OutPitch_Shoulder.STL"/>
+          <mesh filename="package://dvrk_model/meshes/mtm/OutPitch_Shoulder.dae"/>
+        </geometry>
+      </visual>
+      <collision>
+        <geometry>
+          <mesh filename="package://dvrk_model/meshes/mtm/OutPitch_Shoulder.STL"/>
         </geometry>
       </collision>
@@ -83,10 +83,10 @@
       <visual>
         <geometry>
-          <mesh filename="package://irk_model/meshes/mtm/ArmParallel.dae"/>
-        </geometry>
-      </visual>
-      <collision>
-        <geometry>
-          <mesh filename="package://irk_model/meshes/mtm/ArmParallel.STL"/>
+          <mesh filename="package://dvrk_model/meshes/mtm/ArmParallel.dae"/>
+        </geometry>
+      </visual>
+      <collision>
+        <geometry>
+          <mesh filename="package://dvrk_model/meshes/mtm/ArmParallel.STL"/>
         </geometry>
       </collision>
@@ -99,10 +99,10 @@
       <visual>
         <geometry>
-          <mesh filename="package://irk_model/meshes/mtm/ArmParallel1.dae"/>
-        </geometry>
-      </visual>
-      <collision>
-        <geometry>
-          <mesh filename="package://irk_model/meshes/mtm/ArmParallel1.STL"/>
+          <mesh filename="package://dvrk_model/meshes/mtm/ArmParallel1.dae"/>
+        </geometry>
+      </visual>
+      <collision>
+        <geometry>
+          <mesh filename="package://dvrk_model/meshes/mtm/ArmParallel1.STL"/>
         </geometry>
       </collision>
@@ -115,10 +115,10 @@
     <!--   <visual> -->
     <!--     <geometry> -->
-    <!--       <mesh filename="package://irk_model/meshes/mtm/Link.dae"/> -->
+    <!--       <mesh filename="package://dvrk_model/meshes/mtm/Link.dae"/> -->
     <!--     </geometry> -->
     <!--   </visual> -->
     <!--   <collision> -->
     <!--     <geometry> -->
-    <!--       <mesh filename="package://irk_model/meshes/mtm/Link.STL"/> -->
+    <!--       <mesh filename="package://dvrk_model/meshes/mtm/Link.STL"/> -->
     <!--     </geometry> -->
     <!--   </collision> -->
@@ -180,10 +180,10 @@
       <visual>
         <geometry>
-          <mesh filename="package://irk_model/meshes/mtm/WristPlatform.dae"/>
-        </geometry>
-      </visual>
-      <collision>
-        <geometry>
-          <mesh filename="package://irk_model/meshes/mtm/WristPlatform.STL"/>
+          <mesh filename="package://dvrk_model/meshes/mtm/WristPlatform.dae"/>
+        </geometry>
+      </visual>
+      <collision>
+        <geometry>
+          <mesh filename="package://dvrk_model/meshes/mtm/WristPlatform.STL"/>
         </geometry>
       </collision>
@@ -198,10 +198,10 @@
       <visual>
         <geometry>
-          <mesh filename="package://irk_model/meshes/mtm/BottomArm.dae"/>
-        </geometry>
-      </visual>
-      <collision>
-        <geometry>
-          <mesh filename="package://irk_model/meshes/mtm/BottomArm.STL"/>
+          <mesh filename="package://dvrk_model/meshes/mtm/BottomArm.dae"/>
+        </geometry>
+      </visual>
+      <collision>
+        <geometry>
+          <mesh filename="package://dvrk_model/meshes/mtm/BottomArm.STL"/>
         </geometry>
       </collision>
@@ -226,10 +226,10 @@
       <visual>        <!-- defined from CAD file (increased in the y dir by .005-->
         <geometry>
-          <mesh filename="package://irk_model/meshes/mtm/WristPitch.dae"/>
+          <mesh filename="package://dvrk_model/meshes/mtm/WristPitch.dae"/>
         </geometry>
       </visual>
       <collision>        <!-- defined from CAD file (increased in the y dir by .005-->
         <geometry>
-          <mesh filename="package://irk_model/meshes/mtm/WristPitch.STL"/>
+          <mesh filename="package://dvrk_model/meshes/mtm/WristPitch.STL"/>
         </geometry>
       </collision>
@@ -254,10 +254,10 @@
       <visual>
         <geometry>
-          <mesh filename="package://irk_model/meshes/mtm/WristYaw.dae"/>
-        </geometry>
-      </visual>
-      <collision>
-        <geometry>
-          <mesh filename="package://irk_model/meshes/mtm/WristYaw.STL"/>
+          <mesh filename="package://dvrk_model/meshes/mtm/WristYaw.dae"/>
+        </geometry>
+      </visual>
+      <collision>
+        <geometry>
+          <mesh filename="package://dvrk_model/meshes/mtm/WristYaw.STL"/>
         </geometry>
       </collision>
@@ -282,10 +282,10 @@
       <visual>
         <geometry>
-          <mesh filename="package://irk_model/meshes/mtm/WristRoll.dae"/>
-        </geometry>
-      </visual>
-      <collision>
-        <geometry>
-          <mesh filename="package://irk_model/meshes/mtm/WristRoll.STL"/>
+          <mesh filename="package://dvrk_model/meshes/mtm/WristRoll.dae"/>
+        </geometry>
+      </visual>
+      <collision>
+        <geometry>
+          <mesh filename="package://dvrk_model/meshes/mtm/WristRoll.STL"/>
         </geometry>
       </collision>

File: dvrk_model/model/mtm_right.urdf.xacro (robot description, xacro)
@@ -2,5 +2,5 @@
 <robot name="master" xmlns:xacro="http://www.ros.org/wiki/xacro">
   <!-- Macros -->
-  <xacro:include filename="$(find irk_model)/model/mtm.urdf.xacro"/>
+  <xacro:include filename="$(find dvrk_model)/model/mtm.urdf.xacro"/>
   <link name="world"/>
   <xacro:mtm

File: dvrk_model/model/psm.urdf.xacro (robot description, xacro)
@@ -1,4 +1,4 @@
 <?xml version="1.0" encoding="utf-8"?>
-<robot name="irk_psm" xmlns:xacro="http://www.ros.org/wiki/xacro">
+<robot name="dvrk_psm" xmlns:xacro="http://www.ros.org/wiki/xacro">
   <xacro:macro name="psm" params="prefix parent_link xyz rpy">
     <!-- fixed joint -->
@@ -13,5 +13,5 @@
         <origin rpy="1.5708 0 3.1416" xyz="0.039 -0.03888 -0.07879"/>
         <geometry>
-          <mesh filename="package://irk_model/meshes/psm/psm_base.dae"/>
+          <mesh filename="package://dvrk_model/meshes/psm/psm_base.dae"/>
         </geometry>
       </visual>
@@ -31,5 +31,5 @@
         <origin rpy="3.1416 0 1.5708" xyz="0.0125 0 0.1575"/>
         <geometry>
-          <mesh filename="package://irk_model/meshes/psm/outer_yaw.dae"/>
+          <mesh filename="package://dvrk_model/meshes/psm/outer_yaw.dae"/>
         </geometry>
       </visual>
@@ -48,5 +48,5 @@
         <origin rpy="0 0 -0.27129" xyz="0 0 0"/>
         <geometry>
-          <mesh filename="package://irk_model/meshes/psm/outer_pitch_back.dae"/>
+          <mesh filename="package://dvrk_model/meshes/psm/outer_pitch_back.dae"/>
         </geometry>
       </visual>
@@ -66,5 +66,5 @@
         <!-- <origin rpy="0 0 0" xyz="0 0 0"/> -->
         <geometry>
-          <mesh filename="package://irk_model/meshes/psm/outer_pitch_front.dae"/>
+          <mesh filename="package://dvrk_model/meshes/psm/outer_pitch_front.dae"/>
         </geometry>
       </visual>
@@ -83,5 +83,5 @@
         <origin rpy="0 -1.5708 0" xyz="0.009 0 0"/>
         <geometry>
-          <mesh filename="package://irk_model/meshes/psm/outer_pitch_bottom.dae"/>
+          <mesh filename="package://dvrk_model/meshes/psm/outer_pitch_bottom.dae"/>
         </geometry>
       </visual>
@@ -100,5 +100,5 @@
         <origin rpy="0 -1.5708 0" xyz="0.009 0 0"/>
         <geometry>
-          <mesh filename="package://irk_model/meshes/psm/outer_pitch_top.dae"/>
+          <mesh filename="package://dvrk_model/meshes/psm/outer_pitch_top.dae"/>
         </geometry>
       </visual>
@@ -117,5 +117,5 @@
         <origin rpy="0 -1.5708 1.5708" xyz="0.02528 0.429 0"/>
         <geometry>
-          <mesh filename="package://irk_model/meshes/psm/outer_insertion.dae"/>
+          <mesh filename="package://dvrk_model/meshes/psm/outer_insertion.dae"/>
         </geometry>
       </visual>
@@ -134,5 +134,5 @@
         <origin rpy="0 0 1.5708" xyz="0 0 0"/>
         <geometry>
-          <mesh filename="package://irk_model/meshes/psm/tool_main.dae"/>
+          <mesh filename="package://dvrk_model/meshes/psm/tool_main.dae"/>
         </geometry>
       </visual>
@@ -151,5 +151,5 @@
         <origin rpy="0 0 1.5708" xyz="0 0 0"/>
         <geometry>
-          <mesh filename="package://irk_model/meshes/psm/tool_wrist_link.dae"/>
+          <mesh filename="package://dvrk_model/meshes/psm/tool_wrist_link.dae"/>
         </geometry>
       </visual>
@@ -167,5 +167,5 @@
         <origin rpy="1.5708 0 0" xyz="0 0.00401 0"/>
         <geometry>
-          <mesh filename="package://irk_model/meshes/psm/tool_wrist_shaft_link.dae"/>
+          <mesh filename="package://dvrk_model/meshes/psm/tool_wrist_shaft_link.dae"/>
         </geometry>
       </visual>
@@ -185,5 +185,5 @@
         <origin rpy="1.5708 3.1416 0" xyz="0.0051 0.0032 0"/>
         <geometry>
-          <mesh filename="package://irk_model/meshes/psm/tool_wrist_sca_link.dae"/>
+          <mesh filename="package://dvrk_model/meshes/psm/tool_wrist_sca_link.dae"/>
         </geometry>
       </visual>
@@ -203,5 +203,5 @@
         <origin rpy="0 0 0" xyz="0 0 -0.0025"/>
         <geometry>
-          <mesh filename="package://irk_model/meshes/psm/tool_wrist_sca_shaft_link.dae"/>
+          <mesh filename="package://dvrk_model/meshes/psm/tool_wrist_sca_shaft_link.dae"/>
         </geometry>
       </visual>
@@ -221,5 +221,5 @@
         <origin rpy="0 0 0" xyz="0 0 0"/>
         <geometry>
-          <mesh filename="package://irk_model/meshes/psm/tool_wrist_sca_link_2.dae"/>
+          <mesh filename="package://dvrk_model/meshes/psm/tool_wrist_sca_link_2.dae"/>
         </geometry>
       </visual>
@@ -239,5 +239,5 @@
         <origin rpy="0 3.1516 0" xyz="0 0 0"/>
         <geometry>
-          <mesh filename="package://irk_model/meshes/psm/tool_wrist_sca_link_2.dae"/>
+          <mesh filename="package://dvrk_model/meshes/psm/tool_wrist_sca_link_2.dae"/>
         </geometry>
       </visual>

File: dvrk_model/model/psm_jhu.urdf (robot description, URDF)
Before this commit: robot daVinci, 14 links, 13 joints
Links:
- added link world
- link outer_insertion_link: geometry visual mesh filename=package://dvrk_model/meshes/psm/outer_insertion.dae
- link outer_pitch_back_link: geometry visual mesh filename=package://dvrk_model/meshes/psm/outer_pitch_back.dae
- link outer_pitch_bottom_link: geometry visual mesh filename=package://dvrk_model/meshes/psm/outer_pitch_bottom.dae
- link outer_pitch_front_link: geometry visual mesh filename=package://dvrk_model/meshes/psm/outer_pitch_front.dae
- link outer_pitch_top_link: geometry visual mesh filename=package://dvrk_model/meshes/psm/outer_pitch_top.dae
- link outer_yaw_link: geometry visual mesh filename=package://dvrk_model/meshes/psm/outer_yaw.dae
- link psm_base_link: geometry visual mesh filename=package://dvrk_model/meshes/psm/psm_base.dae
- link tool_main_link: geometry visual mesh filename=package://dvrk_model/meshes/psm/tool_main.dae
- link tool_wrist_link: geometry visual mesh filename=package://dvrk_model/meshes/psm/tool_wrist_link.dae
- link tool_wrist_sca_ee_link_1: geometry visual mesh filename=package://dvrk_model/meshes/psm/tool_wrist_sca_link_2.dae
- link tool_wrist_sca_ee_link_2: geometry visual mesh filename=package://dvrk_model/meshes/psm/tool_wrist_sca_link_2.dae
- link tool_wrist_sca_link: geometry visual mesh filename=package://dvrk_model/meshes/psm/tool_wrist_sca_link.dae
- link tool_wrist_sca_shaft_link: geometry visual mesh filename=package://dvrk_model/meshes/psm/tool_wrist_sca_shaft_link.d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
- link tool_wrist_shaft_link: geometry visual mesh filename=package://dvrk_model/meshes/psm/tool_wrist_shaft_link.dae
Joints:
- added joint fixed_joint: type fixed, parent world, child psm_base_link, origin xyz=0.0 0.0 0.0 rpy=0.0 0.0 0.0

File: dvrk_model/model/psm_one.urdf.xacro (robot description, xacro)
@@ -1,6 +1,6 @@
 <?xml version="1.0" ?>
-<robot name="irk_psm" xmlns:xacro="http://www.ros.org/wiki/xacro">
+<robot name="dvrk_psm" xmlns:xacro="http://www.ros.org/wiki/xacro">
   <!-- Macros -->
-  <xacro:include filename="$(find irk_model)/model/psm.urdf.xacro"/>
+  <xacro:include filename="$(find dvrk_model)/model/psm.urdf.xacro"/>
   <link name="world"/>
   <xacro:psm

File: dvrk_model/urdf/daVinci_jhu.urdf (robot description, URDF)
Before this commit: robot irk_psm, 15 links, 14 joints
Links:
- removed link world
- link outer_insertion_link: geometry visual mesh filename=package://dvrk_model/meshes/outer_insertion.dae
- link outer_pitch_back_link: geometry visual mesh filename=package://dvrk_model/meshes/outer_pitch_back.dae
- link outer_pitch_bottom_link: geometry visual mesh filename=package://dvrk_model/meshes/outer_pitch_bottom.dae
- link outer_pitch_front_link: geometry visual mesh filename=package://dvrk_model/meshes/outer_pitch_front.dae
- link outer_pitch_top_link: geometry visual mesh filename=package://dvrk_model/meshes/outer_pitch_top.dae
- link outer_yaw_link: geometry visual mesh filename=package://dvrk_model/meshes/outer_yaw.dae
- link psm_base_link: geometry visual mesh filename=package://dvrk_model/meshes/psm_base.dae
- link tool_main_link: geometry visual mesh filename=package://dvrk_model/meshes/tool_main.dae
- link tool_wrist_link: geometry visual mesh filename=package://dvrk_model/meshes/tool_wrist_link.dae
- link tool_wrist_sca_ee_link_1: geometry visual mesh filename=package://dvrk_model/meshes/tool_wrist_sca_link_2.dae
- link tool_wrist_sca_ee_link_2: geometry visual mesh filename=package://dvrk_model/meshes/tool_wrist_sca_link_2.dae
- link tool_wrist_sca_link: geometry visual mesh filename=package://dvrk_model/meshes/tool_wrist_sca_link.dae
- link tool_wrist_sca_shaft_link: geometry visual mesh filename=package://dvrk_model/meshes/tool_wrist_sca_shaft_link.dae
- link tool_wrist_shaft_link: geometry visual mesh filename=package://dvrk_model/meshes/tool_wrist_shaft_link.dae
Joints:
- removed joint fixed_joint

Commit message: Added transmission tags and custom gazebo controller plugin to mtm.urdf.xacro file

File: dvrk_model/model/mtm.urdf.xacro (robot description, xacro)
@@ -112,20 +112,20 @@
       </inertial>
     </link>
-    <!-- <link name="${prefix}front_parallel_link"> -->
-    <!--   <visual> -->
-    <!--     <geometry> -->
-    <!--       <mesh filename="package://dvrk_model/meshes/mtm/Link.dae"/> -->
-    <!--     </geometry> -->
-    <!--   </visual> -->
-    <!--   <collision> -->
-    <!--     <geometry> -->
-    <!--       <mesh filename="package://dvrk_model/meshes/mtm/Link.STL"/> -->
-    <!--     </geometry> -->
-    <!--   </collision> -->
-    <!--   <inertial> -->
-    <!--     <mass value="0.8"/> -->
-    <!--     <inertia ixx="8.0" ixy="0.0" ixz="0.0" iyy="8.0" iyz="0.0" izz="8.0"/> -->
-    <!--   </inertial>  -->
-    <!-- </link> -->
+     <!--link name="${prefix}front_parallel_link">
+       <visual>
+         <geometry>
+           <mesh filename="package://dvrk_model/meshes/mtm/Link.dae"/>
+         </geometry>
+       </visual>
+       <collision>
+         <geometry>
+           <mesh filename="package://dvrk_model/meshes/mtm/Link.STL"/>
+         </geometry>
+       </collision>
+       <inertial>
+         <mass value="0.8"/>
+         <inertia ixx="8.0" ixy="0.0" ixz="0.0" iyy="8.0" iyz="0.0" izz="8.0"/>
+       </inertial>
+     </link-->
     <joint name="${prefix}shoulder_pitch_joint" type="revolute">
       <parent link="${prefix}outer_yaw_link"/>
@@ -139,7 +139,7 @@
     </joint>
     <joint name="${prefix}shoulder_pitch_parallel_joint" type="revolute">
-      <parent link="${prefix}outer_yaw_link"/>
+      <parent link="${prefix}back_parallel_link"/>
       <child link="${prefix}top_parallel_link"/>
-      <origin rpy="${-PI/2} ${PI} 0" xyz="0 .065 -.19037"/>
+      <origin rpy="0 0 ${-PI/2}" xyz="0 0 0.065"/>
       <axis xyz="0 0 1"/>
       <!--rotates about  x axis-->
@@ -147,14 +147,15 @@
       <limit effort="100.0" lower="${-PI/2}" upper="${PI/2}" velocity="10"/>
       <joint_properties damping="1.0" friction="0.0"/>
-      <mimic joint="${prefix}shoulder_pitch_joint" multiplier="1"/>
-    </joint>
-    <!-- <joint name="${prefix}elbow_pitch_parallel_joint" type="revolute"> -->
-    <!--   <parent link="${prefix}top_parallel_link"/> -->
-    <!--   <child link="${prefix}front_parallel_link"/> -->
-    <!--   <origin rpy="0 0 0" xyz=".1011 0 -0.03"/> -->
-    <!--   <axis xyz="0 0 1"/> -->
-    <!--   <limit effort="100.0" lower="${-PI/4}" upper="${PI/4}" velocity="10"/> -->
-    <!--   <joint_properties damping="1.0" friction="0.0"/> -->
-    <!-- </joint> -->
+      <mimic joint="${prefix}elbow_pitch_joint" multiplier="1"/>
+    </joint>
+    <!--joint name="${prefix}elbow_pitch_parallel_joint" type="revolute">
+       <parent link="${prefix}top_parallel_link"/>
+       <child link="${prefix}front_parallel_link"/>
+       <origin rpy="0 0 0" xyz=".1011 0 -0.03"/>
+       <axis xyz="0 0 1"/>
+       <limit effort="100.0" lower="${-PI/4}" upper="${PI/4}" velocity="10"/>
+       <joint_properties damping="1.0" friction="0.0"/>
+       <mimic joint="${prefix}elbow_pitch_joint" multiplier="-1"/>
+     </joint-->
     <joint name="${prefix}elbow_pitch_joint" type="revolute">
       <parent link="${prefix}back_parallel_link"/>
@@ -297,4 +298,65 @@
       </inertial>
     </link>
+  <transmission name="tran1">
+    <type>transmission_interface/SimpleTransmission</type>
+    <joint name="${prefix}outer_yaw_joint"/>
+    <actuator name="motor1">
+      <hardwareInterface>EffortJointInterface</hardwareInterface>
+      <mechanicalReduction>1</mechanicalReduction>
+    </actuator>
+  </transmission>
+  <transmission name="tran2">
+    <type>transmission_interface/SimpleTransmission</type>
+    <joint name="${prefix}shoulder_pitch_joint"/>
+    <actuator name="motor2">
+      <hardwareInterface>EffortJointInterface</hardwareInterface>
+      <mechanicalReduction>1</mechanicalReduction>
+    </actuator>
+  </transmission>
+  <transmission name="tran3">
+    <type>transmission_interface/SimpleTransmission</type>
+    <joint name="${prefix}elbow_pitch_joint"/>
+    <actuator name="motor3">
+      <hardwareInterface>EffortJointInterface</hardwareInterface>
+      <mechanicalReduction>1</mechanicalReduction>
+    </actuator>
+  </transmission>
+  <transmission name="tran4">
+    <type>transmission_interface/SimpleTransmission</type>
+    <joint name="${prefix}wrist_platform_joint"/>
+    <actuator name="motor4">
+      <hardwareInterface>EffortJointInterface</hardwareInterface>
+      <mechanicalReduction>1</mechanicalReduction>
+    </actuator>
+  </transmission>
+  <transmission name="tran5">
+    <type>transmission_interface/SimpleTransmission</type>
+    <joint name="${prefix}wrist_pitch_joint"/>
+    <actuator name="motor5">
+      <hardwareInterface>EffortJointInterface</hardwareInterface>
+      <mechanicalReduction>1</mechanicalReduction>
+    </actuator>
+  </transmission>
+  <transmission name="tran6">
+    <type>transmission_interface/SimpleTransmission</type>
+    <joint name="${prefix}wrist_yaw_joint"/>
+    <actuator name="motor6">
+      <hardwareInterface>EffortJointInterface</hardwareInterface>
+      <mechanicalReduction>1</mechanicalReduction>
+    </actuator>
+  </transmission>
+  <transmission name="tran7">
+    <type>transmission_interface/SimpleTransmission</type>
+    <joint name="${prefix}wrist_roll_joint"/>
+    <actuator name="motor7">
+      <hardwareInterface>EffortJointInterface</hardwareInterface>
+      <mechanicalReduction>1</mechanicalReduction>
+    </actuator>
+  </transmission>
+  <gazebo>
+    <plugin name="gazebo_ros_control" filename="libgazebo_ros_control.so">
+      <robotNamespace>/mtm</robotNamespace>
+    </plugin>
+  </gazebo>
   </xacro:macro>
 </robot>

Commit message: added fixed base & ee link

File: dvrk_model/model/mtm.urdf.xacro (robot description, xacro)
@@ -297,4 +297,18 @@
       </inertial>
     </link>
+    <!-- add base link to match DVRK manual -->
+    <joint name="${prefix}base" type="fixed">
+      <parent link="${prefix}top_panel"/>
+      <child link="${prefix}base"/>
+      <origin rpy="0 0 0" xyz="0 0 -0.190"/>
+    </joint>
+    <link name="${prefix}base"/>
+    <!-- add ee link to match DVRK manual -->
+    <joint name="${prefix}end_effector" type="fixed">
+      <parent link="${prefix}wrist_roll_link"/>
+      <child link="${prefix}ee_link"/>
+      <origin rpy="0 ${PI} 0" xyz="0 0 0.039"/>
+    </joint>
+    <link name="${prefix}ee_link"/>
   </xacro:macro>
 </robot>
