Commit message: Added motor/transmission plugins for interface with gazebo, does not affect any other functionality of urdf

File: dvrk_model/model/mtm.urdf.xacro (robot description, xacro)
@@ -311,4 +311,74 @@
     </joint>
     <link name="${prefix}ee_link"/>
+    <transmission name="tran1">
+      <type>transmission_interface/SimpleTransmission</type>
+      <joint name="${prefix}outer_yaw_joint"/>
+      <actuator name="motor1">
+        <hardwareInterface>EffortJointInterface</hardwareInterface>
+        <mechanicalReduction>1</mechanicalReduction>
+      </actuator>
+    </transmission>
+    <transmission name="tran2">
+      <type>transmission_interface/SimpleTransmission</type>
+      <joint name="${prefix}shoulder_pitch_joint"/>
+      <actuator name="motor2">
+        <hardwareInterface>EffortJointInterface</hardwareInterface>
+        <mechanicalReduction>1</mechanicalReduction>
+      </actuator>
+    </transmission>
+    <transmission name="tran3">
+      <type>transmission_interface/SimpleTransmission</type>
+      <joint name="${prefix}elbow_pitch_joint"/>
+      <actuator name="motor3">
+        <hardwareInterface>EffortJointInterface</hardwareInterface>
+        <mechanicalReduction>1</mechanicalReduction>
+      </actuator>
+    </transmission>
+    <transmission name="tran4">
+      <type>transmission_interface/SimpleTransmission</type>
+      <joint name="${prefix}wrist_platform_joint"/>
+      <actuator name="motor4">
+        <hardwareInterface>EffortJointInterface</hardwareInterface>
+        <mechanicalReduction>1</mechanicalReduction>
+      </actuator>
+    </transmission>
+    <transmission name="tran5">
+      <type>transmission_interface/SimpleTransmission</type>
+      <joint name="${prefix}wrist_pitch_joint"/>
+      <actuator name="motor5">
+        <hardwareInterface>EffortJointInterface</hardwareInterface>
+        <mechanicalReduction>1</mechanicalReduction>
+      </actuator>
+    </transmission>
+    <transmission name="tran6">
+      <type>transmission_interface/SimpleTransmission</type>
+      <joint name="${prefix}wrist_yaw_joint"/>
+      <actuator name="motor6">
+        <hardwareInterface>EffortJointInterface</hardwareInterface>
+        <mechanicalReduction>1</mechanicalReduction>
+      </actuator>
+    </transmission>
+    <transmission name="tran7">
+      <type>transmission_interface/SimpleTransmission</type>
+      <joint name="${prefix}wrist_roll_joint"/>
+      <actuator name="motor7">
+        <hardwareInterface>EffortJointInterface</hardwareInterface>
+        <mechanicalReduction>1</mechanicalReduction>
+      </actuator>
+    </transmission>
+    <gazebo>
+      <plugin name="gazebo_ros_control" filename="libgazebo_ros_control.so">
+        <robotNamespace>/mtm</robotNamespace>
+      </plugin>
+    </gazebo>
+    <gazebo>
+      <plugin name="force_torque_sensor" filename="libgazebo_ros_f3d.so" >
+        <bodyName>${prefix}bottom_parallel_link</bodyName>
+        <frameName>${prefix}bottom_parallel_link</frameName>
+        <topicName>/force_torque_feedback</topicName>
+        <alwaysOn>true</alwaysOn>
+        <updateRate>100.0</updateRate>
+      </plugin>
+    </gazebo>
   </xacro:macro>
 </robot>

Commit message: added mtm_left_rviz launch file

File: dvrk_model/model/mtm.urdf.xacro (robot description, xacro)
@@ -5,5 +5,4 @@
   <!-- Macro for the da Vinci Master Console -->
   <xacro:macro name="master_console" params="prefix parent_link xyz rpy">
-    <!-- Left MTM -->
     <joint name="${prefix}base_fixed_joint" type="fixed">
       <parent link="${parent_link}"/>
@@ -215,5 +214,5 @@
     <joint name="${prefix}wrist_pitch_joint" type="revolute">
       <parent link="${prefix}wrist_platform_link"/>
-      <child link="${prefix}wrist_pitch_link"/>   <!--rpy="1.57 0 3.14159 " the num .072 & .123 are defined from CAD file -->
+      <child link="${prefix}wrist_pitch_link"/>
       <origin rpy="${-PI/2} 0 0" xyz="0 0 0"/>
       <axis xyz="0 0 1"/>

Commit message: fixed wrist roll link

File: dvrk_model/model/mtm.urdf.xacro (robot description, xacro)
@@ -111,20 +111,4 @@
       </inertial>
     </link>
-    <!-- <link name="${prefix}front_parallel_link"> -->
-    <!--   <visual> -->
-    <!--     <geometry> -->
-    <!--       <mesh filename="package://dvrk_model/meshes/mtm/Link.dae"/> -->
-    <!--     </geometry> -->
-    <!--   </visual> -->
-    <!--   <collision> -->
-    <!--     <geometry> -->
-    <!--       <mesh filename="package://dvrk_model/meshes/mtm/Link.STL"/> -->
-    <!--     </geometry> -->
-    <!--   </collision> -->
-    <!--   <inertial> -->
-    <!--     <mass value="0.8"/> -->
-    <!--     <inertia ixx="8.0" ixy="0.0" ixz="0.0" iyy="8.0" iyz="0.0" izz="8.0"/> -->
-    <!--   </inertial>  -->
-    <!-- </link> -->
     <joint name="${prefix}shoulder_pitch_joint" type="revolute">
       <parent link="${prefix}outer_yaw_link"/>
@@ -271,7 +255,7 @@
       <parent link="${prefix}wrist_yaw_link"/>
       <child link="${prefix}wrist_roll_link"/>  <!-- -.039 & .055 defined from CAD file-->
-      <origin rpy="${-PI/2} ${PI/2} 0" xyz="0 -.039 0"/>
-      <axis xyz="0 0 -1"/>
-      <!--rotates about y axis-->
+      <!-- <origin rpy="${-PI/2} ${PI/2} 0" xyz="0 -.039 0"/> -->
+      <origin rpy="0 ${-PI/2} ${PI/2}" xyz="0 0 0"/>
+      <axis xyz="0 0 1"/>
       <!--limit effort and velocity picked arbitrarily check-->
       <limit effort="100.0" lower="${-1.5*PI}" upper="${1.5*PI}" velocity="10"/>
@@ -280,4 +264,5 @@
     <link name="${prefix}wrist_roll_link">
       <visual>
+        <origin rpy="${PI} 0 0" xyz="0 0 0.039"/>
         <geometry>
           <mesh filename="package://dvrk_model/meshes/mtm/WristRoll.dae"/>
@@ -285,4 +270,5 @@
       </visual>
       <collision>
+        <origin rpy="${PI} 0 0" xyz="0 0 0.039"/>
         <geometry>
           <mesh filename="package://dvrk_model/meshes/mtm/WristRoll.STL"/>
@@ -303,11 +289,4 @@
     </joint>
     <link name="${prefix}base"/>
-    <!-- add ee link to match DVRK manual -->
-    <joint name="${prefix}end_effector" type="fixed">
-      <parent link="${prefix}wrist_roll_link"/>
-      <child link="${prefix}ee_link"/>
-      <origin rpy="0 ${PI} 0" xyz="0 0 0.039"/>
-    </joint>
-    <link name="${prefix}ee_link"/>
     <transmission name="tran1">
       <type>transmission_interface/SimpleTransmission</type>

Commit message: removed base_link, changed joint coordinates to match manual

File: dvrk_model/model/mtm.urdf.xacro (robot description, xacro)
@@ -29,4 +29,5 @@
   <!-- Macro for da Vinci Master Tool Manipulator (MTM) -->
   <xacro:macro name="mtm" params="prefix parent_link xyz rpy">
+    <!-- Joint 0: Fixed to World-->
     <joint name="${prefix}fixed_joint" type="fixed">
       <parent link="${parent_link}"/>
@@ -36,4 +37,5 @@
     <link name="${prefix}top_panel">
       <visual>
+        <origin rpy="0 0 0" xyz="0 0 0.19037"/>
         <geometry>
           <mesh filename="package://dvrk_model/meshes/mtm/Top Panel.dae"/>
@@ -41,4 +43,5 @@
       </visual>
       <collision>
+        <origin rpy="0 0 0" xyz="0 0 0.19037"/>
         <geometry>
           <mesh filename="package://dvrk_model/meshes/mtm/Top Panel.STL"/>
@@ -53,4 +56,5 @@
       </inertial>
     </link>
+    <!-- Joint 1: Outer Yaw -->
     <joint name="${prefix}outer_yaw_joint" type="revolute">
       <parent link="${prefix}top_panel"/>
@@ -65,4 +69,5 @@
     <link name="${prefix}outer_yaw_link">
       <visual>
+        <origin rpy="0 0 0" xyz="0 0 0.19037"/>
         <geometry>
           <mesh filename="package://dvrk_model/meshes/mtm/OutPitch_Shoulder.dae"/>
@@ -70,4 +75,5 @@
       </visual>
       <collision>
+        <origin rpy="0 0 0" xyz="0 0 0.19037"/>
         <geometry>
           <mesh filename="package://dvrk_model/meshes/mtm/OutPitch_Shoulder.STL"/>
@@ -79,50 +85,34 @@
       </inertial>
     </link>
-    <link name="${prefix}back_parallel_link">
-      <visual>
-        <geometry>
-          <mesh filename="package://dvrk_model/meshes/mtm/ArmParallel.dae"/>
-        </geometry>
-      </visual>
-      <collision>
-        <geometry>
-          <mesh filename="package://dvrk_model/meshes/mtm/ArmParallel.STL"/>
-        </geometry>
-      </collision>
-      <inertial>
-        <mass value=".9"/>
-        <inertia ixx="9.0" ixy="0.0" ixz="0.0" iyy="9.0" iyz="0.0" izz="9.0"/>
-      </inertial>
-    </link>
-    <link name="${prefix}top_parallel_link">
-      <visual>
-        <geometry>
-          <mesh filename="package://dvrk_model/meshes/mtm/ArmParallel1.dae"/>
-        </geometry>
-      </visual>
-      <collision>
-        <geometry>
-          <mesh filename="package://dvrk_model/meshes/mtm/ArmParallel1.STL"/>
-        </geometry>
-      </collision>
-      <inertial>
-        <mass value=".5"/>
-        <inertia ixx="5.0" ixy="0.0" ixz="0.0" iyy="5.0" iyz="0.0" izz="5.0"/>
-      </inertial>
-    </link>
+    <!-- Joint 2: Shoulder Pitch -->
     <joint name="${prefix}shoulder_pitch_joint" type="revolute">
       <parent link="${prefix}outer_yaw_link"/>
       <child link="${prefix}back_parallel_link"/>  <!-- xyz= 0 0 -.19037-->
-      <origin rpy="${-PI/2} ${-PI/2} 0" xyz="0 0 -0.19037"/>
-      <axis xyz="0 0 1"/>
-      <!--rotates about  x axis-->
+      <origin rpy="${-PI/2} ${-PI/2} 0" xyz="0 0 0"/>
+      <axis xyz="0 0 1"/>
       <!--limit effort and velocity picked arbitrarily check-->
       <limit effort="100.0" lower="${-PI/4}" upper="${PI/4}" velocity="10"/>
       <joint_properties damping="1.0" friction="0.0"/>
     </joint>
+    <link name="${prefix}back_parallel_link">
+      <visual>
+        <geometry>
+          <mesh filename="package://dvrk_model/meshes/mtm/ArmParallel.dae"/>
+        </geometry>
+      </visual>
+      <collision>
+        <geometry>
+          <mesh filename="package://dvrk_model/meshes/mtm/ArmParallel.STL"/>
+        </geometry>
+      </collision>
+      <inertial>
+        <mass value=".9"/>
+        <inertia ixx="9.0" ixy="0.0" ixz="0.0" iyy="9.0" iyz="0.0" izz="9.0"/>
+      </inertial>
+    </link>
     <joint name="${prefix}shoulder_pitch_parallel_joint" type="revolute">
       <parent link="${prefix}outer_yaw_link"/>
       <child link="${prefix}top_parallel_link"/>
-      <origin rpy="${-PI/2} ${PI} 0" xyz="0 .065 -.19037"/>
+      <origin rpy="${-PI/2} ${-PI/2} 0" xyz="0 0 0"/>
       <axis xyz="0 0 1"/>
       <!--rotates about  x axis-->
@@ -132,26 +122,55 @@
       <mimic joint="${prefix}shoulder_pitch_joint" multiplier="1"/>
     </joint>
-    <!-- <joint name="${prefix}elbow_pitch_parallel_joint" type="revolute"> -->
-    <!--   <parent link="${prefix}top_parallel_link"/> -->
-    <!--   <child link="${prefix}front_parallel_link"/> -->
-    <!--   <origin rpy="0 0 0" xyz=".1011 0 -0.03"/> -->
-    <!--   <axis xyz="0 0 1"/> -->
-    <!--   <limit effort="100.0" lower="${-PI/4}" upper="${PI/4}" velocity="10"/> -->
-    <!--   <joint_properties damping="1.0" friction="0.0"/> -->
-    <!-- </joint> -->
+    <link name="${prefix}top_parallel_link">
+      <visual>
+        <origin rpy="${-PI/2} ${PI} 0" xyz="0 .065 0"/>
+        <geometry>
+          <mesh filename="package://dvrk_model/meshes/mtm/ArmParallel1.dae"/>
+        </geometry>
+      </visual>
+      <collision>
+        <origin rpy="${-PI/2} ${PI} 0" xyz="0 .065 0"/>
+        <geometry>
+          <mesh filename="package://dvrk_model/meshes/mtm/ArmParallel1.STL"/>
+        </geometry>
+      </collision>
+      <inertial>
+        <mass value=".5"/>
+        <inertia ixx="5.0" ixy="0.0" ixz="0.0" iyy="5.0" iyz="0.0" izz="5.0"/>
+      </inertial>
+    </link>
+    <!-- Joint 3: Elbow Pitch -->
     <joint name="${prefix}elbow_pitch_joint" type="revolute">
       <parent link="${prefix}back_parallel_link"/>
       <child link="${prefix}bottom_parallel_link"/>  <!-- xyz= -->
-      <origin rpy="0 0 ${PI/2}" xyz="-.2794 0 0"/>
-      <axis xyz="0 0 1"/>
-      <!--rotates about x axis-->
+      <origin rpy="0 0 ${PI/2}" xyz="-0.2794 0 0"/>
+      <axis xyz="0 0 1"/>
       <!--limit effort and velocity picked arbitrarily check-->
       <limit effort="100.0" lower="${-PI/4}" upper="${PI/4}" velocity="10"/>
       <joint_properties damping="1.0" friction="0.0"/>
     </joint>
+    <link name="${prefix}bottom_parallel_link">
+      <visual>
+        <geometry>
+          <mesh filename="package://dvrk_model/meshes/mtm/BottomArm.dae"/>
+        </geometry>
+      </visual>
+      <collision>
+        <geometry>
+          <mesh filename="package://dvrk_model/meshes/mtm/BottomArm.STL"/>
+        </geometry>
+      </collision>
+      <inertial>
+        <mass value="0.8"/>
+        <inertia ixx="0.1" ixy="0.0" ixz="0.0"
+                 iyy="0.1" iyz="0.0"
+                 izz="0.1"/>
+      </inertial>
+    </link>
+    <!-- Joint 4: Platform -->
     <joint name="${prefix}wrist_platform_joint" type="revolute">
       <parent link="${prefix}bottom_parallel_link"/>
-      <child link="${prefix}wrist_platform_link"/>  <!-- -.348 & -.02746 defined from MTMDaVinci paper and  added -.01 from original to align, -0.02746 defined from CAD file-->
-      <origin rpy="${PI/2} 0 0" xyz="-0.3645 -0.156 0.0"/>
+      <child link="${prefix}wrist_platform_link"/>
+      <origin rpy="${PI/2} 0 0" xyz="-0.3645 -0.1506 0.0"/>
       <axis xyz="0 0 1"/>
       <!--rotates about z axis-->
@@ -178,22 +197,5 @@
       </inertial>
     </link>
-    <link name="${prefix}bottom_parallel_link">
-      <visual>
-        <geometry>
-          <mesh filename="package://dvrk_model/meshes/mtm/BottomArm.dae"/>
-        </geometry>
-      </visual>
-      <collision>
-        <geometry>
-          <mesh filename="package://dvrk_model/meshes/mtm/BottomArm.STL"/>
-        </geometry>
-      </collision>
-      <inertial>
-        <mass value="0.8"/>
-        <inertia ixx="0.1" ixy="0.0" ixz="0.0"
-                           iyy="0.1" iyz="0.0"
-                                     izz="0.1"/>
-      </inertial>
-    </link>
+    <!-- Joint 5: Wrist Pitch -->
     <joint name="${prefix}wrist_pitch_joint" type="revolute">
       <parent link="${prefix}wrist_platform_link"/>
@@ -201,5 +203,4 @@
       <origin rpy="${-PI/2} 0 0" xyz="0 0 0"/>
       <axis xyz="0 0 1"/>
-      <!--rotates about x axis-->
       <!--limit effort and velocity picked arbitrarily check-->
       <limit effort="100.0" lower="${-PI/2}" upper="${PI}" velocity="10"/>
@@ -224,4 +225,5 @@
       </inertial>
     </link>
+    <!-- Joint 6: Wrist Yaw-->
     <joint name="${prefix}wrist_yaw_joint" type="revolute">
       <parent link="${prefix}wrist_pitch_link"/>
@@ -252,4 +254,5 @@
       </inertial>
     </link>
+    <!-- Joint 7: Wrist Roll -->
     <joint name="${prefix}wrist_roll_joint" type="revolute">
       <parent link="${prefix}wrist_yaw_link"/>
@@ -282,11 +285,4 @@
       </inertial>
     </link>
-    <!-- add base link to match DVRK manual -->
-    <joint name="${prefix}base" type="fixed">
-      <parent link="${prefix}top_panel"/>
-      <child link="${prefix}base"/>
-      <origin rpy="0 0 0" xyz="0 0 -0.190"/>
-    </joint>
-    <link name="${prefix}base"/>
     <transmission name="tran1">
       <type>transmission_interface/SimpleTransmission</type>

Commit message: fixed top_yaw_link

File: dvrk_model/model/mtm.urdf.xacro (robot description, xacro)
@@ -69,5 +69,5 @@
     <link name="${prefix}outer_yaw_link">
       <visual>
-        <origin rpy="0 0 0" xyz="0 0 0.19037"/>
+        <origin rpy="0 0 0" xyz="0.025 0 0.19037"/>
         <geometry>
           <mesh filename="package://dvrk_model/meshes/mtm/OutPitch_Shoulder.dae"/>
@@ -75,5 +75,5 @@
       </visual>
       <collision>
-        <origin rpy="0 0 0" xyz="0 0 0.19037"/>
+        <origin rpy="0 0 0" xyz="0.025 0 0.19037"/>
         <geometry>
           <mesh filename="package://dvrk_model/meshes/mtm/OutPitch_Shoulder.STL"/>
@@ -124,5 +124,5 @@
     <link name="${prefix}top_parallel_link">
       <visual>
-        <origin rpy="${-PI/2} ${PI} 0" xyz="0 .065 0"/>
+        <origin rpy="0 0 ${-PI/2}" xyz="0 0 0.065"/>
         <geometry>
           <mesh filename="package://dvrk_model/meshes/mtm/ArmParallel1.dae"/>
@@ -130,5 +130,5 @@
       </visual>
       <collision>
-        <origin rpy="${-PI/2} ${PI} 0" xyz="0 .065 0"/>
+        <origin rpy="0 0 0" xyz="0 0 0"/>
         <geometry>
           <mesh filename="package://dvrk_model/meshes/mtm/ArmParallel1.STL"/>
