Commit message: fixed MTML arm urdf

File: dvrk_model/model/mtm.urdf.xacro (robot description, xacro)
@@ -15,15 +15,17 @@
   </xacro:macro>
   <!-- Macros for left and right MTMs -->
-  <xacro:macro name="left_mtm" params="prefix parent_link">
+  <xacro:macro name="mtm_left" params="prefix parent_link xyz rpy">
     <xacro:mtm
-      prefix="${prefix}left_"
-      parent_link="${parent_link}"
-      xyz="-0.25 0.0 1.0" rpy="0.0 0.0 ${30/180*PI}"/>
+        prefix="${prefix}left_"
+        parent_link="${parent_link}"
+        xyz="${xyz}" rpy="${rpy}"/>
+    <xacro:mtm_platform_left prefix="${prefix}left_"/>
   </xacro:macro>
-  <xacro:macro name="right_mtm" params="prefix parent_link">
+  <xacro:macro name="mtm_right" params="prefix parent_link xyz rpy">
     <xacro:mtm
       prefix="${prefix}right_"
       parent_link="${parent_link}"
-      xyz="0.25 0.0 1.0" rpy="0.0 0.0 0.0"/>
+      xyz="${xyz}" rpy="${rpy}"/>
+    <xacro:mtm_platform_right prefix="${prefix}right_"/>
   </xacro:macro>
   <!-- Macro for da Vinci Master Tool Manipulator (MTM) -->
@@ -168,121 +170,4 @@
       </inertial>
     </link>
-    <!-- Joint 4: Platform -->
-    <joint name="${prefix}wrist_platform_joint" type="revolute">
-      <parent link="${prefix}bottom_parallel_link"/>
-      <child link="${prefix}wrist_platform_link"/>
-      <origin rpy="${PI/2} 0 0" xyz="-0.3645 -0.1506 0.0"/>
-      <axis xyz="0 0 1"/>
-      <!--rotates about z axis-->
-      <!--limit effort and velocity picked arbitrarily check-->
-      <limit effort="100.0" lower="${-60/180*PI}" upper="${245/180*PI}" velocity="10"/>
-      <joint_properties damping="1.0" friction="0.0"/>
-    </joint>
-    <link name="${prefix}wrist_platform_link">
-      <visual>
-        <geometry>
-          <mesh filename="package://dvrk_model/meshes/mtm/WristPlatform.dae"/>
-        </geometry>
-      </visual>
-      <collision>
-        <geometry>
-          <mesh filename="package://dvrk_model/meshes/mtm/WristPlatform.STL"/>
-        </geometry>
-      </collision>
-      <inertial>
-        <mass value="0.4"/>
-        <inertia ixx="0.1" ixy="0.0" ixz="0.0"
-                           iyy="0.1" iyz="0.0"
-                                     izz="0.1"/>
-      </inertial>
-    </link>
-    <!-- Joint 5: Wrist Pitch -->
-    <joint name="${prefix}wrist_pitch_joint" type="revolute">
-      <parent link="${prefix}wrist_platform_link"/>
-      <child link="${prefix}wrist_pitch_link"/>
-      <origin rpy="${-PI/2} 0 0" xyz="0 0 0"/>
-      <axis xyz="0 0 1"/>
-      <!--limit effort and velocity picked arbitrarily check-->
-      <limit effort="100.0" lower="${-PI/2}" upper="${PI}" velocity="10"/>
-      <joint_properties damping="1.0" friction="0.0"/>
-    </joint>
-    <link name="${prefix}wrist_pitch_link">
-      <visual>        <!-- defined from CAD file (increased in the y dir by .005-->
-        <geometry>
-          <mesh filename="package://dvrk_model/meshes/mtm/WristPitch.dae"/>
-        </geometry>
-      </visual>
-      <collision>        <!-- defined from CAD file (increased in the y dir by .005-->
-        <geometry>
-          <mesh filename="package://dvrk_model/meshes/mtm/WristPitch.STL"/>
-        </geometry>
-      </collision>
-      <inertial>
-        <mass value="0.2"/>
-        <inertia ixx="0.1" ixy="0.0" ixz="0.0"
-                           iyy="0.1" iyz="0.0"
-                                     izz="0.1"/>
-      </inertial>
-    </link>
-    <!-- Joint 6: Wrist Yaw-->
-    <joint name="${prefix}wrist_yaw_joint" type="revolute">
-      <parent link="${prefix}wrist_pitch_link"/>
-      <child link="${prefix}wrist_yaw_link"/>    <!--  defined from CAD file-->
-      <origin rpy="${PI/2} ${-PI/2} 0" xyz="0 0 0"/>
-      <axis xyz="0 0 1"/>
-      <!--rotates about z axis-->
-      <!--limit effort and velocity picked arbitrarily check-->
-      <limit effort="100.0"  lower="${-PI/4}" upper="${PI/4}" velocity="10"/>
-      <joint_properties damping="1.0" friction="0.0"/>
-    </joint>
-    <link name="${prefix}wrist_yaw_link">
-      <visual>
-        <geometry>
-          <mesh filename="package://dvrk_model/meshes/mtm/WristYaw.dae"/>
-        </geometry>
-      </visual>
-      <collision>
-        <geometry>
-          <mesh filename="package://dvrk_model/meshes/mtm/WristYaw.STL"/>
-        </geometry>
-      </collision>
-      <inertial>
-        <mass value="0.2"/>
-        <inertia ixx="0.1" ixy="0.0" ixz="0.0"
-                           iyy="0.1" iyz="0.0"
-                                     izz="0.1"/>
-      </inertial>
-    </link>
-    <!-- Joint 7: Wrist Roll -->
-    <joint name="${prefix}wrist_roll_joint" type="revolute">
-      <parent link="${prefix}wrist_yaw_link"/>
-      <child link="${prefix}wrist_roll_link"/>  <!-- -.039 & .055 defined from CAD file-->
-      <!-- <origin rpy="${-PI/2} ${PI/2} 0" xyz="0 -.039 0"/> -->
-      <origin rpy="0 ${-PI/2} ${PI/2}" xyz="0 0 0"/>
-      <axis xyz="0 0 1"/>
-      <!--limit effort and velocity picked arbitrarily check-->
-      <limit effort="100.0" lower="${-1.5*PI}" upper="${1.5*PI}" velocity="10"/>
-      <joint_properties damping="1.0" friction="0.0"/>
-    </joint>
-    <link name="${prefix}wrist_roll_link">
-      <visual>
-        <origin rpy="${PI} 0 0" xyz="0 0 0.039"/>
-        <geometry>
-          <mesh filename="package://dvrk_model/meshes/mtm/WristRoll.dae"/>
-        </geometry>
-      </visual>
-      <collision>
-        <origin rpy="${PI} 0 0" xyz="0 0 0.039"/>
-        <geometry>
-          <mesh filename="package://dvrk_model/meshes/mtm/WristRoll.STL"/>
-        </geometry>
-      </collision>
-      <inertial>
-        <mass value="0.1"/>
-        <inertia ixx="0.1" ixy="0.0" ixz="0.0"
-                           iyy="0.1" iyz="0.0"
-                                     izz="0.1"/>
-      </inertial>
-    </link>
     <transmission name="tran1">
       <type>transmission_interface/SimpleTransmission</type>
@@ -305,36 +190,4 @@
       <joint name="${prefix}elbow_pitch_joint"/>
       <actuator name="motor3">
-        <hardwareInterface>EffortJointInterface</hardwareInterface>
-        <mechanicalReduction>1</mechanicalReduction>
-      </actuator>
-    </transmission>
-    <transmission name="tran4">
-      <type>transmission_interface/SimpleTransmission</type>
-      <joint name="${prefix}wrist_platform_joint"/>
-      <actuator name="motor4">
-        <hardwareInterface>EffortJointInterface</hardwareInterface>
-        <mechanicalReduction>1</mechanicalReduction>
-      </actuator>
-    </transmission>
-    <transmission name="tran5">
-      <type>transmission_interface/SimpleTransmission</type>
-      <joint name="${prefix}wrist_pitch_joint"/>
-      <actuator name="motor5">
-        <hardwareInterface>EffortJointInterface</hardwareInterface>
-        <mechanicalReduction>1</mechanicalReduction>
-      </actuator>
-    </transmission>
-    <transmission name="tran6">
-      <type>transmission_interface/SimpleTransmission</type>
-      <joint name="${prefix}wrist_yaw_joint"/>
-      <actuator name="motor6">
-        <hardwareInterface>EffortJointInterface</hardwareInterface>
-        <mechanicalReduction>1</mechanicalReduction>
-      </actuator>
-    </transmission>
-    <transmission name="tran7">
-      <type>transmission_interface/SimpleTransmission</type>
-      <joint name="${prefix}wrist_roll_joint"/>
-      <actuator name="motor7">
         <hardwareInterface>EffortJointInterface</hardwareInterface>
         <mechanicalReduction>1</mechanicalReduction>
@@ -356,3 +209,311 @@
     </gazebo>
   </xacro:macro>
+  <!-- Macro for dVRK MTM Platform Right -->
+  <xacro:macro name="mtm_platform_right" params="prefix">
+    <!-- Joint 4: Platform -->
+    <joint name="${prefix}wrist_platform_joint" type="revolute">
+      <parent link="${prefix}bottom_parallel_link"/>
+      <child link="${prefix}wrist_platform_link"/>
+      <origin rpy="${PI/2} 0 0" xyz="-0.3645 -0.1506 0.0"/>
+      <axis xyz="0 0 1"/>
+      <!--rotates about z axis-->
+      <!--limit effort and velocity picked arbitrarily check-->
+      <limit effort="100.0" lower="${-60/180*PI}" upper="${245/180*PI}" velocity="10"/>
+      <joint_properties damping="1.0" friction="0.0"/>
+    </joint>
+    <link name="${prefix}wrist_platform_link">
+      <visual>
+        <geometry>
+          <mesh filename="package://dvrk_model/meshes/mtm/WristPlatform.dae"/>
+        </geometry>
+      </visual>
+      <collision>
+        <geometry>
+          <mesh filename="package://dvrk_model/meshes/mtm/WristPlatform.STL"/>
+        </geometry>
+      </collision>
+      <inertial>
+        <mass value="0.4"/>
+        <inertia ixx="0.1" ixy="0.0" ixz="0.0"
+                 iyy="0.1" iyz="0.0"
+                 izz="0.1"/>
+      </inertial>
+    </link>
+    <!-- Joint 5: Wrist Pitch -->
+    <joint name="${prefix}wrist_pitch_joint" type="revolute">
+      <parent link="${prefix}wrist_platform_link"/>
+      <child link="${prefix}wrist_pitch_link"/>
+      <origin rpy="${-PI/2} 0 0" xyz="0 0 0"/>
+      <axis xyz="0 0 1"/>
+      <!--limit effort and velocity picked arbitrarily check-->
+      <limit effort="100.0" lower="${-PI/2}" upper="${PI}" velocity="10"/>
+      <joint_properties damping="1.0" friction="0.0"/>
+    </joint>
+    <link name="${prefix}wrist_pitch_link">
+      <visual>        <!-- defined from CAD file (increased in the y dir by .005-->
+        <geometry>
+          <mesh filename="package://dvrk_model/meshes/mtm/WristPitch.dae"/>
+        </geometry>
+      </visual>
+      <collision>        <!-- defined from CAD file (increased in the y dir by .005-->
+        <geometry>
+          <mesh filename="package://dvrk_model/meshes/mtm/WristPitch.STL"/>
+        </geometry>
+      </collision>
+      <inertial>
+        <mass value="0.2"/>
+        <inertia ixx="0.1" ixy="0.0" ixz="0.0"
+                 iyy="0.1" iyz="0.0"
+                 izz="0.1"/>
+      </inertial>
+    </link>
+    <!-- Joint 6: Wrist Yaw-->
+    <joint name="${prefix}wrist_yaw_joint" type="revolute">
+      <parent link="${prefix}wrist_pitch_link"/>
+      <child link="${prefix}wrist_yaw_link"/>    <!--  defined from CAD file-->
+      <origin rpy="${PI/2} ${-PI/2} 0" xyz="0 0 0"/>
+      <axis xyz="0 0 1"/>
+      <!--rotates about z axis-->
+      <!--limit effort and velocity picked arbitrarily check-->
+      <limit effort="100.0"  lower="${-PI/4}" upper="${PI/4}" velocity="10"/>
+      <joint_properties damping="1.0" friction="0.0"/>
+    </joint>
+    <link name="${prefix}wrist_yaw_link">
+      <visual>
+        <geometry>
+          <mesh filename="package://dvrk_model/meshes/mtm/WristYaw.dae"/>
+        </geometry>
+      </visual>
+      <collision>
+        <geometry>
+          <mesh filename="package://dvrk_model/meshes/mtm/WristYaw.STL"/>
+        </geometry>
+      </collision>
+      <inertial>
+        <mass value="0.2"/>
+        <inertia ixx="0.1" ixy="0.0" ixz="0.0"
+                 iyy="0.1" iyz="0.0"
+                 izz="0.1"/>
+      </inertial>
+    </link>
+    <!-- Joint 7: Wrist Roll -->
+    <joint name="${prefix}wrist_roll_joint" type="revolute">
+      <parent link="${prefix}wrist_yaw_link"/>
+      <child link="${prefix}wrist_roll_link"/>  <!-- -.039 & .055 defined from CAD file-->
+      <!-- <origin rpy="${-PI/2} ${PI/2} 0" xyz="0 -.039 0"/> -->
+      <origin rpy="0 ${-PI/2} ${PI/2}" xyz="0 0 0"/>
+      <axis xyz="0 0 1"/>
+      <!--limit effort and velocity picked arbitrarily check-->
+      <limit effort="100.0" lower="${-1.5*PI}" upper="${1.5*PI}" velocity="10"/>
+      <joint_properties damping="1.0" friction="0.0"/>
+    </joint>
+    <link name="${prefix}wrist_roll_link">
+      <visual>
+        <origin rpy="${PI} 0 0" xyz="0 0 0.039"/>
+        <geometry>
+          <mesh filename="package://dvrk_model/meshes/mtm/WristRoll.dae"/>
+        </geometry>
+      </visual>
+      <collision>
+        <origin rpy="${PI} 0 0" xyz="0 0 0.039"/>
+        <geometry>
+          <mesh filename="package://dvrk_model/meshes/mtm/WristRoll.STL"/>
+        </geometry>
+      </collision>
+      <inertial>
+        <mass value="0.1"/>
+        <inertia ixx="0.1" ixy="0.0" ixz="0.0"
+                 iyy="0.1" iyz="0.0"
+                 izz="0.1"/>
+      </inertial>
+    </link>
+    <transmission name="tran4">
+      <type>transmission_interface/SimpleTransmission</type>
+      <joint name="${prefix}wrist_platform_joint"/>
+      <actuator name="motor4">
+        <hardwareInterface>EffortJointInterface</hardwareInterface>
+        <mechanicalReduction>1</mechanicalReduction>
+      </actuator>
+    </transmission>
+    <transmission name="tran5">
+      <type>transmission_interface/SimpleTransmission</type>
+      <joint name="${prefix}wrist_pitch_joint"/>
+      <actuator name="motor5">
+        <hardwareInterface>EffortJointInterface</hardwareInterface>
+        <mechanicalReduction>1</mechanicalReduction>
+      </actuator>
+    </transmission>
+    <transmission name="tran6">
+      <type>transmission_interface/SimpleTransmission</type>
+      <joint name="${prefix}wrist_yaw_joint"/>
+      <actuator name="motor6">
+        <hardwareInterface>EffortJointInterface</hardwareInterface>
+        <mechanicalReduction>1</mechanicalReduction>
+      </actuator>
+    </transmission>
+    <transmission name="tran7">
+      <type>transmission_interface/SimpleTransmission</type>
+      <joint name="${prefix}wrist_roll_joint"/>
+      <actuator name="motor7">
+        <hardwareInterface>EffortJointInterface</hardwareInterface>
+        <mechanicalReduction>1</mechanicalReduction>
+      </actuator>
+    </transmission>
+  </xacro:macro>
+  <!-- Macro for dVRK MTM Platform Left -->
+  <xacro:macro name="mtm_platform_left" params="prefix">
+    <!-- Joint 4: Platform -->
+    <joint name="${prefix}wrist_platform_joint" type="revolute">
+      <parent link="${prefix}bottom_parallel_link"/>
+      <child link="${prefix}wrist_platform_link"/>
+      <origin rpy="${PI/2} 0 0" xyz="-0.3645 -0.1506 0.0"/>
+      <axis xyz="0 0 1"/>
+      <!--rotates about z axis-->
+      <!--limit effort and velocity picked arbitrarily check-->
+      <limit effort="100.0" lower="${-60/180*PI}" upper="${245/180*PI}" velocity="10"/>
+      <joint_properties damping="1.0" friction="0.0"/>
+    </joint>
+    <link name="${prefix}wrist_platform_link">
+      <visual>
+        <origin rpy="0 0 ${PI}" xyz="0.0 0.0 0.0"/>
+        <geometry>
+          <mesh filename="package://dvrk_model/meshes/mtm/WristPlatform.dae"/>
+        </geometry>
+      </visual>
+      <collision>
+        <origin rpy="0 0 ${PI}" xyz="0.0 0.0 0.0"/>
+        <geometry>
+          <mesh filename="package://dvrk_model/meshes/mtm/WristPlatform.STL"/>
+        </geometry>
+      </collision>
+      <inertial>
+        <mass value="0.4"/>
+        <inertia ixx="0.1" ixy="0.0" ixz="0.0"
+                 iyy="0.1" iyz="0.0"
+                 izz="0.1"/>
+      </inertial>
+    </link>
+    <!-- Joint 5: Wrist Pitch -->
+    <joint name="${prefix}wrist_pitch_joint" type="revolute">
+      <parent link="${prefix}wrist_platform_link"/>
+      <child link="${prefix}wrist_pitch_link"/>
+      <origin rpy="${-PI/2} 0 0" xyz="0 0 0"/>
+      <axis xyz="0 0 1"/>
+      <!--limit effort and velocity picked arbitrarily check-->
+      <limit effort="100.0" lower="${-PI/2}" upper="${PI}" velocity="10"/>
+      <joint_properties damping="1.0" friction="0.0"/>
+    </joint>
+    <link name="${prefix}wrist_pitch_link">
+      <visual>        <!-- defined from CAD file (increased in the y dir by .005-->
+        <origin rpy="0 ${PI} 0" xyz="0.0 0.0 0.0"/>
+        <geometry>
+          <mesh filename="package://dvrk_model/meshes/mtm/WristPitch.dae"/>
+        </geometry>
+      </visual>
+      <collision>        <!-- defined from CAD file (increased in the y dir by .005-->
+        <origin rpy="0 ${PI} 0" xyz="0.0 0.0 0.0"/>
+        <geometry>
+          <mesh filename="package://dvrk_model/meshes/mtm/WristPitch.STL"/>
+        </geometry>
+      </collision>
+      <inertial>
+        <mass value="0.2"/>
+        <inertia ixx="0.1" ixy="0.0" ixz="0.0"
+                 iyy="0.1" iyz="0.0"
+                 izz="0.1"/>
+      </inertial>
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
File: dvrk_model/model/mtm_left.urdf.xacro (robot description, xacro)
@@ -4,6 +4,6 @@
   <xacro:include filename="$(find dvrk_model)/model/mtm.urdf.xacro"/>
   <link name="world"/>
-  <xacro:mtm
-      prefix="left_"
+  <xacro:mtm_left
+      prefix=""
       parent_link="world"
       xyz="-0.25 0.0 1.0" rpy="0.0 0.0 0.0"/>

File: dvrk_model/model/mtm_right.urdf.xacro (robot description, xacro)
@@ -4,6 +4,6 @@
   <xacro:include filename="$(find dvrk_model)/model/mtm.urdf.xacro"/>
   <link name="world"/>
-  <xacro:mtm
-      prefix="right_"
+  <xacro:mtm_right
+      prefix=""
       parent_link="world"
       xyz="0.25 0.0 1.0" rpy="0.0 0.0 0.0"/>
