Commit message: fixed ecm yaw pitch

File: dvrk_model/model/ecm.urdf.xacro (robot description, xacro)
@@ -6,12 +6,19 @@
   <xacro:macro name="ecm" params="prefix parent_link xyz rpy">
     <!-- Joint 0: Fixed to World-->
-    <joint name="${prefix}fixed_joint" type="fixed">
+    <joint name="${prefix}_setup_fixed_joint" type="fixed">
       <parent link="${parent_link}"/>
-      <child link="${prefix}setup_link"/>
+      <child link="${prefix}_setup_base_link"/>
       <origin rpy="${rpy}" xyz="${xyz}"/>
     </joint>
-    <link name="${prefix}setup_link">
-      <visual>
-        <origin rpy="${PI} 0 0" xyz="0 0 0"/>
+    <link name="${prefix}_setup_base_link"/>
+    <joint name="${prefix}_setup_tip_joint" type="fixed">
+      <parent link="${prefix}_setup_base_link"/>
+      <child link="${prefix}_setup_link"/>
+      <origin rpy="-0.87046370379 0 -${PI/2}" xyz="0.91324 -0.02111 0.03166"/>
+      <axis xyz="0 0 1"/>
+    </joint>
+    <link name="${prefix}_setup_link">
+      <visual>
+        <origin rpy="0 0 0" xyz="0 0 0"/>
         <geometry>
           <mesh filename="package://dvrk_model/meshes/ecm/Endo_Arm.STL"/>
@@ -20,5 +27,5 @@
       </visual>
       <collision>
-        <origin rpy="${PI} 0 0" xyz="0 0 0"/>
+        <origin rpy="0 0 0" xyz="0 0 0"/>
         <geometry>
           <mesh filename="package://dvrk_model/meshes/ecm/Endo_Arm.STL"/>
@@ -26,9 +33,16 @@
       </collision>
     </link>
+    <!-- Joint 0: Fixed to Setup Joint-->
+    <joint name="${prefix}_fixed_joint" type="fixed">
+      <parent link="${prefix}_setup_link"/>
+      <child link="${prefix}_base_link"/>
+      <origin rpy="0 0 0" xyz="0 0.603 0"/>
+    </joint>
+    <link name="${prefix}_base_link"/>
     <!-- Joint 1: Outer Yaw -->
     <joint name="${prefix}_yaw_joint" type="revolute">
-      <parent link="${prefix}setup_link"/>
+      <parent link="${prefix}_base_link"/>
       <child link="${prefix}_yaw_link"/>
-      <origin rpy="0 -0.700332623 0" xyz="0.91324 -0.02111 0.03166"/>
+      <origin rpy="0 -${PI/2} ${PI/2}" xyz="0 0 0"/>
       <axis xyz="0 0 1"/>
       <!--rotates about z axis-->
@@ -39,5 +53,5 @@
     <link name="${prefix}_yaw_link">
       <visual>
-        <origin rpy="0 0 -${PI/2}" xyz="0.0 0 0.0"/>
+        <origin rpy="0 0 -${PI/2}" xyz="0.0 0 0.603"/>
         <geometry>
           <mesh filename="package://dvrk_model/meshes/ecm/Endo_Link_5.STL"/>
@@ -46,5 +60,5 @@
       </visual>
       <collision>
-        <origin rpy="0 0 -${PI/2}" xyz="0.0 0 0.0"/>
+        <origin rpy="0 0 -${PI/2}" xyz="0.0 0 0.603"/>
         <geometry>
           <mesh filename="package://dvrk_model/meshes/ecm/Endo_Link_5.STL"/>
@@ -55,9 +69,18 @@
     <joint name="${prefix}_pitch_joint" type="revolute">
       <parent link="${prefix}_yaw_link"/>
+      <child link="${prefix}_pitch_link"/>
+      <origin rpy="-${PI/2} -${PI/2} 0" xyz="0 0 0"/>
+      <axis xyz="0 0 1"/>
+      <limit effort="100.0" lower="${-PI/4}" upper="${PI*65/180}" velocity="10"/>
+      <joint_properties damping="1.0" friction="0.0"/>
+    </joint>
+    <link name="${prefix}_pitch_link"/>
+    <joint name="${prefix}_pitch_joint_0" type="continuous">
+      <parent link="${prefix}_yaw_link"/>
       <child link="${prefix}_pitch_link_1"/>
-      <origin rpy="-${PI/2} -${PI/2} 0" xyz="0 0 -0.225"/>
-      <axis xyz="0 0 1"/>
-      <limit effort="100.0" lower="${-PI/4}" upper="${PI*65/180}" velocity="10"/>
-      <joint_properties damping="1.0" friction="0.0"/>
+      <origin rpy="-${PI/2} -${PI/2} 0" xyz="0 0 0.378"/>
+      <axis xyz="0 0 1"/>
+      <joint_properties damping="1.0" friction="0.0"/>
+      <mimic joint="${prefix}_pitch_joint" multiplier="1"/>
     </joint>
     <link name="${prefix}_pitch_link_1">

Commit message: ecm frames matches DH/manual

File: dvrk_model/model/ecm.urdf.xacro (robot description, xacro)
@@ -159,7 +159,7 @@
     <!-- Joint 3: Insertion -->
     <joint name="${prefix}_insertion_joint" type="prismatic">
-      <parent link="${prefix}_pitch_link_3"/>
+      <parent link="${prefix}_pitch_link"/>
       <child link="${prefix}_insertion_link"/>
-      <origin rpy="${PI/2} 0 0" xyz="-0.09382 0.15 0"/>
+      <origin rpy="${PI/2} 0 0" xyz="0 0.3822 0"/>
       <axis xyz="0 0 1"/>
       <joint_properties damping="1.0" friction="0.0"/>
@@ -168,5 +168,5 @@
     <link name="${prefix}_insertion_link">
       <visual>
-        <origin rpy="0 0 -${PI/2}" xyz="0.0 0 0"/>
+        <origin rpy="0 0 -${PI/2}" xyz="0.0 0 -0.015"/>
         <geometry>
           <mesh filename="package://dvrk_model/meshes/ecm/Endo_Link_8.STL"/>
@@ -175,5 +175,5 @@
       </visual>
       <collision>
-        <origin rpy="0 0 -${PI/2}" xyz="0.0 0 0"/>
+        <origin rpy="0 0 -${PI/2}" xyz="0.0 0 -0.015"/>
         <geometry>
           <mesh filename="package://dvrk_model/meshes/ecm/Endo_Link_8.STL"/>
@@ -185,5 +185,5 @@
       <parent link="${prefix}_insertion_link"/>
       <child link="${prefix}_roll_link"/>
-      <origin rpy="0 0 0" xyz="0 0 0"/>
+      <origin rpy="0 0 0" xyz="0 0 0.3829"/>
       <axis xyz="0 0 1"/>
       <joint_properties damping="1.0" friction="0.0"/>
@@ -192,5 +192,5 @@
     <link name="${prefix}_roll_link">
       <visual>
-        <origin rpy="0 0 ${PI/2}" xyz="0.0 0 0"/>
+        <origin rpy="0 0 ${PI/2}" xyz="0.0 0 -0.3979"/>
         <geometry>
           <mesh filename="package://dvrk_model/meshes/ecm/EndoScope.STL"/>
@@ -199,5 +199,5 @@
       </visual>
       <collision>
-        <origin rpy="0 0 ${PI/2}" xyz="0.0 0 0"/>
+        <origin rpy="0 0 ${PI/2}" xyz="0.0 0 -0.3979"/>
         <geometry>
           <mesh filename="package://dvrk_model/meshes/ecm/EndoScope.STL"/>

Commit message: fix base_joint

File: dvrk_model/model/ecm.urdf.xacro (robot description, xacro)
@@ -4,10 +4,10 @@
   <xacro:include filename="$(find dvrk_model)/model/common.urdf.xacro"/>
   <link name="world"/>
-  <joint name="base_joint" type="fixed">
+  <joint name="setup_joint" type="fixed">
     <parent link="world"/>
-    <child link="ecm_base_link"/>
+    <child link="ecm_setup_link"/>
     <origin rpy="0 0 0" xyz="0 0 1"/>
   </joint>
-  <link name="ecm_base_link">
+  <link name="ecm_setup_link">
     <visual>
       <origin rpy="0 0 0" xyz="0 0 0"/>
@@ -31,10 +31,15 @@
     </inertial>
   </link>
+  <joint name="ecm_base_joint" type="fixed">
+    <parent link="ecm_setup_link"/>
+    <child link="ecm_base_link"/>
+    <origin rpy="-0.870463703366 0 -1.5707963267948966" xyz="0.92717 0 -0.12728"/>
+  </joint>
+  <link name="ecm_base_link"></link>
   <joint name="ecm_yaw_joint" type="revolute">
     <parent link="ecm_base_link"/>
     <child link="ecm_yaw_link"/>
-    <!--fix xyz value-->
-    <origin rpy="-0.870463703366 0 -1.5707963267948966" xyz="0.92717 0 -0.12728"/>
-    <axis xyz="0 1 0"/>
+    <origin rpy="1.5707963267948966 -1.5707963267948966 0" xyz="0 0 0"/>
+    <axis xyz="0 0 1"/>
     <limit effort="50.0" lower="-1.5707963267948966" upper="1.5707963267948966" velocity="2"/>
     <joint_properties damping="1.0" friction="0.0"/>

Commit message: update joint limit

File: dvrk_model/model/ecm.urdf.xacro (robot description, xacro)
@@ -40,12 +40,12 @@
     <parent link="ecm_base_link"/>
     <child link="ecm_yaw_link"/>
-    <origin rpy="1.5707963267948966 -1.5707963267948966 0" xyz="0 0 0"/>
-    <axis xyz="0 0 1"/>
-    <limit effort="50.0" lower="-1.5707963267948966" upper="1.5707963267948966" velocity="2"/>
+    <origin rpy="${PI/2} ${-PI/2} 0" xyz="0 0 0"/>
+    <axis xyz="0 0 1"/>
+    <limit effort="50.0" lower="${-PI/2}" upper="${PI/2}" velocity="2"/>
     <joint_properties damping="1.0" friction="0.0"/>
   </joint>
   <link name="ecm_yaw_link">
     <visual>
-      <origin rpy="0 0 0" xyz="0 0 0"/>
+      <origin rpy="-1.5707963267948966 0 -1.5707963267948966" xyz="0 0 0"/>
       <geometry>
         <mesh filename="package://dvrk_model/meshes/ecm/ecm_yaw_link.STL"/>
@@ -56,5 +56,5 @@
     </visual>
     <collision>
-      <origin rpy="0 0 0" xyz="0 0 0"/>
+      <origin rpy="-1.5707963267948966 0 -1.5707963267948966" xyz="0 0 0"/>
       <geometry>
         <mesh filename="package://dvrk_model/meshes/ecm/ecm_yaw_link.STL"/>
@@ -62,5 +62,5 @@
     </collision>
     <inertial>
-      <origin rpy="0 0 0" xyz="0 0 0"/>
+      <origin rpy="-1.5707963267948966 0 -1.5707963267948966" xyz="0 0 0"/>
       <mass value=".9"/>
       <inertia ixx="9.0" ixy="0.0" ixz="0.0" iyy="9.0" iyz="0.0" izz="9.0"/>
@@ -70,7 +70,7 @@
     <parent link="ecm_yaw_link"/>
     <child link="ecm_pitch_link_1"/>
-    <origin rpy="1.570796326794896 0 -1.570796326794896" xyz="0 0.225 0"/>
-    <axis xyz="0 0 1"/>
-    <limit effort="50.0" lower="-0.785398163397" upper="0.785398163397" velocity="2"/>
+    <origin rpy="-1.570796326794896 -1.570796326794896 0" xyz="0 0 -0.225"/>
+    <axis xyz="0 0 1"/>
+    <limit effort="50.0" lower="${-PI/4}" upper="${PI*65/180}" velocity="2"/>
     <joint_properties damping="1.0" friction="0.0"/>
   </joint>
@@ -164,5 +164,5 @@
     <origin rpy="1.5707963267948966 0 0" xyz="-0.08805 0.14212563 0"/>
     <axis xyz="0 0 1"/>
-    <limit effort="1000.0" lower="0" upper="0.3020714143" velocity="2"/>
+    <limit effort="1000.0" lower="0" upper="0.235" velocity="2"/>
     <joint_properties damping="1.0" friction="0.0"/>
   </joint>
@@ -195,5 +195,5 @@
     <origin rpy="0 0 0" xyz="0 0 0.383"/>
     <axis xyz="0 0 1"/>
-    <limit effort="50.0" lower="-1.57079632" upper="1.57079632" velocity="2"/>
+    <limit effort="50.0" lower="${-PI/2}" upper="${PI/2}" velocity="2"/>
     <joint_properties damping="1.0" friction="0.0"/>
   </joint>

Commit message: fix pitch joint

File: dvrk_model/model/ecm.urdf.xacro (robot description, xacro)
@@ -100,5 +100,5 @@
     <parent link="ecm_pitch_link_1"/>
     <child link="ecm_pitch_link_2"/>
-    <origin rpy="0 0 0.198187435043" xyz="0.05512992 0.274519 0"/>
+    <origin rpy="0 0 0" xyz="0.05512992 0.274519 0"/>
     <axis xyz="0 0 1"/>
     <limit effort="50.0" lower="-0.785398163397" upper="0.785398163397" velocity="2"/>

Commit message: relocate roll/pitch/yaw origin

File: dvrk_model/model/ecm.urdf.xacro (robot description, xacro)
@@ -40,5 +40,5 @@
     <parent link="ecm_base_link"/>
     <child link="ecm_yaw_link"/>
-    <origin rpy="${PI/2} ${-PI/2} 0" xyz="0 0 0"/>
+    <origin rpy="${PI/2} ${-PI/2} 0" xyz="0 0.565 0"/>
     <axis xyz="0 0 1"/>
     <limit effort="50.0" lower="${-PI/2}" upper="${PI/2}" velocity="2"/>
@@ -47,5 +47,5 @@
   <link name="ecm_yaw_link">
     <visual>
-      <origin rpy="-1.5707963267948966 0 -1.5707963267948966" xyz="0 0 0"/>
+      <origin rpy="-1.5707963267948966 0 -1.5707963267948966" xyz="0 0 0.565"/>
       <geometry>
         <mesh filename="package://dvrk_model/meshes/ecm/ecm_yaw_link.STL"/>
@@ -56,5 +56,5 @@
     </visual>
     <collision>
-      <origin rpy="-1.5707963267948966 0 -1.5707963267948966" xyz="0 0 0"/>
+      <origin rpy="-1.5707963267948966 0 -1.5707963267948966" xyz="0 0 0.565"/>
       <geometry>
         <mesh filename="package://dvrk_model/meshes/ecm/ecm_yaw_link.STL"/>
@@ -62,20 +62,30 @@
     </collision>
     <inertial>
-      <origin rpy="-1.5707963267948966 0 -1.5707963267948966" xyz="0 0 0"/>
-      <mass value=".9"/>
-      <inertia ixx="9.0" ixy="0.0" ixz="0.0" iyy="9.0" iyz="0.0" izz="9.0"/>
-    </inertial>
-  </link>
+      <origin rpy="-1.5707963267948966 0 -1.5707963267948966" xyz="0 0 0.565"/>
+      <mass value=".9"/>
+      <inertia ixx="9.0" ixy="0.0" ixz="0.0" iyy="9.0" iyz="0.0" izz="9.0"/>
+    </inertial>
+  </link>
+  <joint name="ecm_pitch_joint" type="revolute">
+    <parent link="ecm_yaw_link"/>
+    <child link="ecm_pitch_link"/>
+    <origin rpy="-1.570796326794896 -1.570796326794896 0" xyz="0 0 0"/>
+    <axis xyz="0 0 1"/>
+    <limit effort="50.0" lower="${-PI/4}" upper="${PI*65/180}" velocity="2"/>
+    <joint_properties damping="1.0" friction="0.0"/>
+  </joint>
+  <link name="ecm_pitch_link"></link>
   <joint name="ecm_pitch_joint_1" type="revolute">
     <parent link="ecm_yaw_link"/>
     <child link="ecm_pitch_link_1"/>
-    <origin rpy="-1.570796326794896 -1.570796326794896 0" xyz="0 0 -0.225"/>
+    <origin rpy="-1.570796326794896 -1.570796326794896 0" xyz="0 0 0.34"/>
     <axis xyz="0 0 1"/>
     <limit effort="50.0" lower="${-PI/4}" upper="${PI*65/180}" velocity="2"/>
     <joint_properties damping="1.0" friction="0.0"/>
+    <mimic joint="ecm_pitch_joint" multiplier="1"/>
   </joint>
   <link name="ecm_pitch_link_1">
     <visual>
-      <origin rpy="0 0 -0.198187435043" xyz="0 0 0"/>
+      <origin rpy="0 0 -0.3198923" xyz="0 0 0"/>
       <geometry>
         <mesh filename="package://dvrk_model/meshes/ecm/ecm_pitch_link_1.STL"/>
@@ -86,5 +96,5 @@
     </visual>
     <collision>
-      <origin rpy="0 0 -0.198187435043" xyz="0 0 0"/>
+      <origin rpy="0 0 -0.3198923" xyz="0 0 0"/>
       <geometry>
         <mesh filename="package://dvrk_model/meshes/ecm/ecm_pitch_link_1.STL"/>
@@ -92,5 +102,5 @@
     </collision>
     <inertial>
-      <origin rpy="0 0 -0.198187435043" xyz="0 0 0"/>
+      <origin rpy="0 0 -0.3198923" xyz="0 0 0"/>
       <mass value=".9"/>
       <inertia ixx="9.0" ixy="0.0" ixz="0.0" iyy="9.0" iyz="0.0" izz="9.0"/>
@@ -100,9 +110,9 @@
     <parent link="ecm_pitch_link_1"/>
     <child link="ecm_pitch_link_2"/>
-    <origin rpy="0 0 0" xyz="0.05512992 0.274519 0"/>
+    <origin rpy="0 0 0" xyz="0.08805 0.2657954 0"/>
     <axis xyz="0 0 1"/>
     <limit effort="50.0" lower="-0.785398163397" upper="0.785398163397" velocity="2"/>
     <joint_properties damping="1.0" friction="0.0"/>
-    <mimic joint="ecm_pitch_joint_1" multiplier="-1"/>
+    <mimic joint="ecm_pitch_joint" multiplier="-1"/>
   </joint>
   <link name="ecm_pitch_link_2">
@@ -135,5 +145,5 @@
     <limit effort="50.0" lower="-0.785398163397" upper="0.785398163397" velocity="2"/>
     <joint_properties damping="1.0" friction="0.0"/>
-    <mimic joint="ecm_pitch_joint_1" multiplier="1"/>
+    <mimic joint="ecm_pitch_joint" multiplier="1"/>
   </joint>
   <link name="ecm_pitch_link_3">
@@ -159,13 +169,55 @@
     </inertial>
   </link>
+  <joint name="ecm_roll_joint" type="revolute">
+    <parent link="ecm_pitch_link"/>
+    <child link="ecm_roll_link"/>
+    <!--fix z value-->
+    <origin rpy="${PI/2} 0 0" xyz="0 0 0"/>
+    <axis xyz="0 0 1"/>
+    <limit effort="50.0" lower="${-PI/2}" upper="${PI/2}" velocity="2"/>
+    <joint_properties damping="1.0" friction="0.0"/>
+  </joint>
+  <link name="ecm_roll_link"></link>
   <joint name="ecm_insertion_joint" type="prismatic">
-    <parent link="ecm_pitch_link_3"/>
+    <parent link="ecm_roll_link"/>
     <child link="ecm_insertion_link"/>
-    <origin rpy="1.5707963267948966 0 0" xyz="-0.08805 0.14212563 0"/>
-    <axis xyz="0 0 1"/>
-    <limit effort="1000.0" lower="0" upper="0.235" velocity="2"/>
+    <origin rpy="0 0 0" xyz="0 0 0"/>
+    <axis xyz="0 0 1"/>
+    <limit effort="1000.0" lower="-0.02492103" upper="0.210078977" velocity="2"/>
     <joint_properties damping="1.0" friction="0.0"/>
   </joint>
   <link name="ecm_insertion_link">
+    <visual>
+      <origin rpy="0 0 ${PI}" xyz="0 0 0"/>
+      <geometry>
+        <mesh filename="package://dvrk_model/meshes/ecm/ecm_roll_link.STL"/>
+      </geometry>
+      <material name="DaVinciDarkGray">
+        <color rgba="${DaVinciDarkGray}"/>
+      </material>
+    </visual>
+    <collision>
+      <origin rpy="0 0 ${PI}" xyz="0 0 0"/>
+      <geometry>
+        <mesh filename="package://dvrk_model/meshes/ecm/ecm_roll_link.STL"/>
+      </geometry>
+    </collision>
+    <inertial>
+      <origin rpy="0 0 ${PI}" xyz="0 0 0"/>
+      <mass value=".9"/>
+      <inertia ixx="9.0" ixy="0.0" ixz="0.0" iyy="9.0" iyz="0.0" izz="9.0"/>
+    </inertial>
+  </link>
+  <!--This part is for the attached link on the endoscope, only for visualization purpose-->
+  <joint name="ecm_insertion_joint_attach" type="revolute">
+    <parent link="ecm_insertion_link"/>
+    <child link="ecm_insertion_link_attach"/>
+    <origin rpy="0 0 0" xyz="0 0 -0.383"/>
+    <axis xyz="0 0 1"/>
+    <limit effort="50.0" lower="${-PI/2}" upper="${PI/2}" velocity="2"/>
+    <joint_properties damping="1.0" friction="0.0"/>
+    <mimic joint="ecm_roll_joint" multiplier="-1"/>
+  </joint>
+  <link name="ecm_insertion_link_attach">
     <visual>
       <origin rpy="3.1415926 0 0" xyz="0 0 0"/>
@@ -189,34 +241,3 @@
     </inertial>
   </link>
-  <joint name="ecm_roll_joint" type="revolute">
-    <parent link="ecm_insertion_link"/>
-    <child link="ecm_roll_link"/>
-    <!--fix z value-->
-    <origin rpy="0 0 0" xyz="0 0 0.383"/>
-    <axis xyz="0 0 1"/>
-    <limit effort="50.0" lower="${-PI/2}" upper="${PI/2}" velocity="2"/>
-    <joint_properties damping="1.0" friction="0.0"/>
-  </joint>
-  <link name="ecm_roll_link">
-    <visual>
-      <origin rpy="0 0 0" xyz="0 0 0"/>
-      <geometry>
-        <mesh filename="package://dvrk_model/meshes/ecm/ecm_roll_link.STL"/>
-      </geometry>
-      <material name="DaVinciDarkGray">
-        <color rgba="${DaVinciDarkGray}"/>
-      </material>
-    </visual>
-    <collision>
-      <origin rpy="0 0 0" xyz="0 0 0"/>
-      <geometry>
-        <mesh filename="package://dvrk_model/meshes/ecm/ecm_roll_link.STL"/>
-      </geometry>
-    </collision>
-    <inertial>
-      <origin rpy="0 0 0" xyz="0 0 0"/>
-      <mass value=".9"/>
-      <inertia ixx="9.0" ixy="0.0" ixz="0.0" iyy="9.0" iyz="0.0" izz="9.0"/>
-    </inertial>
-  </link>
 </robot>
