Commit message: psm.tool.caudier.urdf.xacro now uses meshes in dvrk_model

File: dvrk_model/model/psm.tool.caudier.urdf.xacro (robot description, xacro)
@@ -15,5 +15,5 @@
         <origin rpy="0.00 -1.5708 0.0" xyz="-0.0024 0.00 0.000"/>
         <geometry>
-          <mesh filename="package://dvrk_nri_model/meshes/tool_wrist_caudier_link_1.stl"/>
+          <mesh filename="package://dvrk_model/meshes/psm/tool_wrist_caudier_link_1.stl"/>
         </geometry>
         <material name="gray"><color rgba="0.5 0.5 0.9 1.0"/></material>
@@ -22,5 +22,5 @@
         <origin rpy="0.00 -1.5708 0.0" xyz="-0.0024 0.00 0.000"/>
         <geometry>
-          <mesh filename="package://dvrk_nri_model/meshes/tool_wrist_caudier_link_1.stl"/>
+          <mesh filename="package://dvrk_model/meshes/psm/tool_wrist_caudier_link_1.stl"/>
         </geometry>
       </collision>
@@ -39,5 +39,5 @@
         <origin rpy="0.00 1.5708 0.0" xyz="0.0 -0.0002 0.000"/>
         <geometry>
-          <mesh filename="package://dvrk_nri_model/meshes/tool_wrist_caudier_link_1_shaft.stl"/>
+          <mesh filename="package://dvrk_model/meshes/psm/tool_wrist_caudier_link_1_shaft.stl"/>
         </geometry>
         <material name="gray"><color rgba="0.5 0.5 0.9 1.0"/></material>
@@ -46,5 +46,5 @@
         <origin rpy="0.00 1.5708 0.0" xyz="0.0 0.00 0.000"/>
         <geometry>
-          <mesh filename="package://dvrk_nri_model/meshes/tool_wrist_caudier_link_1_shaft.stl"/>
+          <mesh filename="package://dvrk_model/meshes/psm/tool_wrist_caudier_link_1_shaft.stl"/>
         </geometry>
       </collision>
@@ -63,5 +63,5 @@
         <origin rpy="0.0 0 0.0" xyz="0 0 0.00195"/>
         <geometry>
-          <mesh filename="package://dvrk_nri_model/meshes/tool_wrist_caudier_link_2_left.stl"/>
+          <mesh filename="package://dvrk_model/meshes/psm/tool_wrist_caudier_link_2_left.stl"/>
         </geometry>
       </visual>
@@ -69,5 +69,5 @@
         <origin rpy="0.0 0 0.0" xyz="0 0 0.00195"/>
         <geometry>
-          <mesh filename="package://dvrk_nri_model/meshes/tool_wrist_caudier_link_2_left.stl"/>
+          <mesh filename="package://dvrk_model/meshes/psm/tool_wrist_caudier_link_2_left.stl"/>
         </geometry>
       </collision>
@@ -87,5 +87,5 @@
         <origin rpy="0 0 -3.1415926" xyz="0 0 0.00195"/>
         <geometry>
-          <mesh filename="package://dvrk_nri_model/meshes/tool_wrist_caudier_link_2_right.stl"/>
+          <mesh filename="package://dvrk_model/meshes/psm/tool_wrist_caudier_link_2_right.stl"/>
         </geometry>
       </visual>
@@ -93,5 +93,5 @@
         <origin rpy="0 0 -3.1415926" xyz="0 0 0.00195"/>
         <geometry>
-          <mesh filename="package://dvrk_nri_model/meshes/tool_wrist_caudier_link_2_right.stl"/>
+          <mesh filename="package://dvrk_model/meshes/psm/tool_wrist_caudier_link_2_right.stl"/>
         </geometry>
       </collision>

Commit message: changed joint names in urdf files and fixed in python script

File: dvrk_model/model/psm.tool.caudier.urdf.xacro (robot description, xacro)
@@ -51,5 +51,5 @@
     </link>
     <!-- joint 6-1: Outer open angle 1 -->
-    <joint name="${prefix}outer_wrist_open_angle_joint_left" type="revolute">
+    <joint name="${prefix}outer_wrist_open_angle_joint" type="revolute">
       <parent link="${prefix}tool_wrist_caudier_link_shaft"/>
       <child link="${prefix}tool_wrist_caudier_link_2_left"/>
@@ -74,5 +74,5 @@
     </link>
     <!-- joint 6-2: Outer open angle 2  -->
-    <joint name="${prefix}outer_wrist_open_angle_joint_right" type="revolute">
+    <joint name="${prefix}outer_wrist_open_angle_joint_mimic" type="revolute">
       <parent link="${prefix}tool_wrist_caudier_link_shaft"/>
       <child link="${prefix}tool_wrist_caudier_link_2_right"/>
@@ -80,5 +80,5 @@
       <origin rpy="3.1415926 0 0" xyz="0 0 0"/>
       <limit lower="0" upper="1.5707" velocity=".4" effort="1000"/>
-      <mimic joint="${prefix}outer_wrist_open_angle_joint_left" multiplier="1"/>
+      <mimic joint="${prefix}outer_wrist_open_angle_joint" multiplier="1"/>
     </joint>
     <!-- link 6-2: Outer open angle link 2 -->

File: dvrk_model/model/psm.tool.sca.urdf.xacro (robot description, xacro)
@@ -41,5 +41,5 @@
     </link>
     <!-- joint 7-1: Outer open angle 1  -->
-    <joint name="${prefix}outer_wrist_open_angle_joint_1" type="revolute">
+    <joint name="${prefix}outer_wrist_open_angle_joint" type="revolute">
       <parent link="${prefix}tool_wrist_sca_shaft_link"/>
       <child link="${prefix}tool_wrist_sca_ee_link_1"/>
@@ -58,5 +58,5 @@
     </link>
     <!-- joint 7-2: Outer open angle 2   -->
-    <joint name="${prefix}outer_wrist_open_angle_joint_2" type="revolute">
+    <joint name="${prefix}outer_wrist_open_angle_joint_mimic" type="revolute">
       <parent link="${prefix}tool_wrist_sca_shaft_link"/>
       <child link="${prefix}tool_wrist_sca_ee_link_2"/>
@@ -64,5 +64,5 @@
       <origin rpy="0 0 0" xyz="0 0 0"/>
       <limit lower="-1.5707" upper="1.5707" velocity=".4" effort="1000"/>
-      <mimic joint="${prefix}outer_wrist_open_angle_joint_1" multiplier="-1"/>
+      <mimic joint="${prefix}outer_wrist_open_angle_joint" multiplier="-1"/>
     </joint>
     <!-- link 7-2: Outer open angle link 2 -->

Commit message: Removing SI conversion(joints alraedy in SI); Adding end effector link to match with forward kinematics

File: dvrk_model/model/psm.tool.caudier.urdf.xacro (robot description, xacro)
@@ -97,4 +97,14 @@
       </collision>
     </link>
+    <!-- joint 6-3:   -->
+    <joint name="${prefix}tool_wrist_caudier_ee_joint" type="revolute">
+      <parent link="${prefix}tool_wrist_caudier_link_shaft"/>
+      <child link="${prefix}tool_wrist_caudier_ee_link"/>
+      <axis xyz="0 0 1"/>
+      <origin rpy="0.0 1.5708 1.5708" xyz="0 0 0"/>
+      <limit lower="-1.5707" upper="1.5707" velocity=".4" effort="1000"/>
+    </joint>
+    <!-- link 6-3:  -->
+    <link name="${prefix}tool_wrist_caudier_ee_link" />
   </xacro:macro>
 </robot>
