Commit message: Updated urdf/launch and rviz files to use dvrk_ros topic names (i.e. PSM1, PSM2, ...), fixed urdf for PSM tool jaw angles, renamed joint names in urdf files to match dvrk_ros topics, removed requirement on dvrk_joint_publisher ROS package (was used to add joint names, now come from PID XML config), use same stl file for both sides of caudiere jaw

File: dvrk_model/model/MTML.urdf.xacro (robot description, xacro)
@@ -4,7 +4,7 @@
   <xacro:include filename="$(find dvrk_model)/model/mtm.urdf.xacro"/>
   <link name="world"/>
-  <xacro:mtm_right
-      prefix=""
+  <xacro:mtm_left
+      prefix="$(arg prefix)"
       parent_link="world"
-      xyz="0.25 0.0 1.0" rpy="0.0 0.0 0.0"/>
+      xyz="-0.25 0.0 1.0" rpy="0.0 0.0 0.0"/>
 </robot>

File: dvrk_model/model/MTMR.urdf.xacro (robot description, xacro)
@@ -4,7 +4,7 @@
   <xacro:include filename="$(find dvrk_model)/model/mtm.urdf.xacro"/>
   <link name="world"/>
-  <xacro:mtm_left
-      prefix=""
+  <xacro:mtm_right
+      prefix="$(arg prefix)"
       parent_link="world"
-      xyz="-0.25 0.0 1.0" rpy="0.0 0.0 0.0"/>
+      xyz="0.25 0.0 1.0" rpy="0.0 0.0 0.0"/>
 </robot>

File: dvrk_model/model/PSM1.urdf.xacro (robot description, xacro)
@@ -4,7 +4,7 @@
   <xacro:include filename="$(find dvrk_model)/model/psm.urdf.xacro"/>
   <link name="world"/>
-  <xacro:psm_caudier
-      prefix="two_"
+  <xacro:psm_sca
+      prefix="$(arg prefix)"
       parent_link="world"
-      xyz="0.25 0.0 0.5" rpy="0.0 0.0 -3.1415926"/>
+      xyz="-0.25 0.0 0.5" rpy="0.0 0.0 3.1415926"/>
 </robot>

File: dvrk_model/model/PSM2.urdf.xacro (robot description, xacro)
@@ -4,7 +4,7 @@
   <xacro:include filename="$(find dvrk_model)/model/psm.urdf.xacro"/>
   <link name="world"/>
-  <xacro:psm
-      prefix="three_"
+  <xacro:psm_caudier
+      prefix="$(arg prefix)"
       parent_link="world"
-      xyz="0.50 0.0 0.5" rpy="0.0 0.0 -3.1415926"/>
+      xyz="0.25 0.0 0.5" rpy="0.0 0.0 -3.1415926"/>
 </robot>

File: dvrk_model/model/PSM3.urdf.xacro (robot description, xacro)
@@ -4,7 +4,7 @@
   <xacro:include filename="$(find dvrk_model)/model/psm.urdf.xacro"/>
   <link name="world"/>
-  <xacro:psm_sca
-      prefix="one_"
-      parent_link="world"
-      xyz="-0.25 0.0 0.5" rpy="0.0 0.0 3.1415926"/>
+  <xacro:psm_caudier
+    prefix="$(arg prefix)"
+    parent_link="world"
+    xyz="0.50 0.0 0.5" rpy="0.0 0.0 -3.1415926"/>
 </robot>

File: dvrk_model/model/mtm.urdf.xacro (robot description, xacro)
@@ -5,5 +5,5 @@
   <!-- Macro for the da Vinci Master Console -->
   <xacro:macro name="master_console" params="prefix parent_link xyz rpy">
-    <joint name="${prefix}base_fixed_joint" type="fixed">
+    <joint name="base_fixed" type="fixed">
       <parent link="${parent_link}"/>
       <child link="${prefix}master_base_link"/>
@@ -17,20 +17,20 @@
   <xacro:macro name="mtm_left" params="prefix parent_link xyz rpy">
     <xacro:mtm
-        prefix="${prefix}left_"
+        prefix="${prefix}"
         parent_link="${parent_link}"
         xyz="${xyz}" rpy="${rpy}"/>
-    <xacro:mtm_platform_left prefix="${prefix}left_"/>
+    <xacro:mtm_platform_left prefix="${prefix}"/>
   </xacro:macro>
   <xacro:macro name="mtm_right" params="prefix parent_link xyz rpy">
     <xacro:mtm
-      prefix="${prefix}right_"
+      prefix="${prefix}"
       parent_link="${parent_link}"
       xyz="${xyz}" rpy="${rpy}"/>
-    <xacro:mtm_platform_right prefix="${prefix}right_"/>
+    <xacro:mtm_platform_right prefix="${prefix}"/>
   </xacro:macro>
   <!-- Macro for da Vinci Master Tool Manipulator (MTM) -->
   <xacro:macro name="mtm" params="prefix parent_link xyz rpy">
     <!-- Joint 0: Fixed to World-->
-    <joint name="${prefix}fixed_joint" type="fixed">
+    <joint name="fixed" type="fixed">
       <parent link="${parent_link}"/>
       <child link="${prefix}top_panel"/>
@@ -59,5 +59,5 @@
     </link>
     <!-- Joint 1: Outer Yaw -->
-    <joint name="${prefix}outer_yaw_joint" type="revolute">
+    <joint name="outer_yaw" type="revolute">
       <parent link="${prefix}top_panel"/>
       <child link="${prefix}outer_yaw_link"/>
@@ -88,5 +88,5 @@
     </link>
     <!-- Joint 2: Shoulder Pitch -->
-    <joint name="${prefix}shoulder_pitch_joint" type="revolute">
+    <joint name="shoulder_pitch" type="revolute">
       <parent link="${prefix}outer_yaw_link"/>
       <child link="${prefix}back_parallel_link"/>  <!-- xyz= 0 0 -.19037-->
@@ -113,5 +113,5 @@
       </inertial>
     </link>
-    <joint name="${prefix}shoulder_pitch_parallel_joint" type="revolute">
+    <joint name="shoulder_pitch_parallel" type="revolute">
       <parent link="${prefix}outer_yaw_link"/>
       <child link="${prefix}top_parallel_link"/>
@@ -122,5 +122,5 @@
       <limit effort="100.0" lower="${-PI/2}" upper="${PI/2}" velocity="10"/>
       <joint_properties damping="1.0" friction="0.0"/>
-      <mimic joint="${prefix}shoulder_pitch_joint" multiplier="1"/>
+      <mimic joint="shoulder_pitch" multiplier="1"/>
     </joint>
     <link name="${prefix}top_parallel_link">
@@ -143,5 +143,5 @@
     </link>
     <!-- Joint 3: Elbow Pitch -->
-    <joint name="${prefix}elbow_pitch_joint" type="revolute">
+    <joint name="elbow_pitch" type="revolute">
       <parent link="${prefix}back_parallel_link"/>
       <child link="${prefix}bottom_parallel_link"/>  <!-- xyz= -->
@@ -172,5 +172,5 @@
     <transmission name="tran1">
       <type>transmission_interface/SimpleTransmission</type>
-      <joint name="${prefix}outer_yaw_joint"/>
+      <joint name="outer_yaw"/>
       <actuator name="motor1">
         <hardwareInterface>EffortJointInterface</hardwareInterface>
@@ -180,5 +180,5 @@
     <transmission name="tran2">
       <type>transmission_interface/SimpleTransmission</type>
-      <joint name="${prefix}shoulder_pitch_joint"/>
+      <joint name="shoulder_pitch"/>
       <actuator name="motor2">
         <hardwareInterface>EffortJointInterface</hardwareInterface>
@@ -188,5 +188,5 @@
     <transmission name="tran3">
       <type>transmission_interface/SimpleTransmission</type>
-      <joint name="${prefix}elbow_pitch_joint"/>
+      <joint name="elbow_pitch"/>
       <actuator name="motor3">
         <hardwareInterface>EffortJointInterface</hardwareInterface>
@@ -212,5 +212,5 @@
   <xacro:macro name="mtm_platform_right" params="prefix">
     <!-- Joint 4: Platform -->
-    <joint name="${prefix}wrist_platform_joint" type="revolute">
+    <joint name="wrist_platform" type="revolute">
       <parent link="${prefix}bottom_parallel_link"/>
       <child link="${prefix}wrist_platform_link"/>
@@ -241,5 +241,5 @@
     </link>
     <!-- Joint 5: Wrist Pitch -->
-    <joint name="${prefix}wrist_pitch_joint" type="revolute">
+    <joint name="wrist_pitch" type="revolute">
       <parent link="${prefix}wrist_platform_link"/>
       <child link="${prefix}wrist_pitch_link"/>
@@ -269,5 +269,5 @@
     </link>
     <!-- Joint 6: Wrist Yaw-->
-    <joint name="${prefix}wrist_yaw_joint" type="revolute">
+    <joint name="wrist_yaw" type="revolute">
       <parent link="${prefix}wrist_pitch_link"/>
       <child link="${prefix}wrist_yaw_link"/>    <!--  defined from CAD file-->
@@ -298,5 +298,5 @@
     </link>
     <!-- Joint 7: Wrist Roll -->
-    <joint name="${prefix}wrist_roll_joint" type="revolute">
+    <joint name="wrist_roll" type="revolute">
       <parent link="${prefix}wrist_yaw_link"/>
       <child link="${prefix}wrist_roll_link"/>  <!-- -.039 & .055 defined from CAD file-->
@@ -330,5 +330,5 @@
     <transmission name="tran4">
       <type>transmission_interface/SimpleTransmission</type>
-      <joint name="${prefix}wrist_platform_joint"/>
+      <joint name="wrist_platform"/>
       <actuator name="motor4">
         <hardwareInterface>EffortJointInterface</hardwareInterface>
@@ -338,5 +338,5 @@
     <transmission name="tran5">
       <type>transmission_interface/SimpleTransmission</type>
-      <joint name="${prefix}wrist_pitch_joint"/>
+      <joint name="wrist_pitch"/>
       <actuator name="motor5">
         <hardwareInterface>EffortJointInterface</hardwareInterface>
@@ -346,5 +346,5 @@
     <transmission name="tran6">
       <type>transmission_interface/SimpleTransmission</type>
-      <joint name="${prefix}wrist_yaw_joint"/>
+      <joint name="wrist_yaw"/>
       <actuator name="motor6">
         <hardwareInterface>EffortJointInterface</hardwareInterface>
@@ -354,5 +354,5 @@
     <transmission name="tran7">
       <type>transmission_interface/SimpleTransmission</type>
-      <joint name="${prefix}wrist_roll_joint"/>
+      <joint name="wrist_roll"/>
       <actuator name="motor7">
         <hardwareInterface>EffortJointInterface</hardwareInterface>
@@ -364,5 +364,5 @@
   <xacro:macro name="mtm_platform_left" params="prefix">
     <!-- Joint 4: Platform -->
-    <joint name="${prefix}wrist_platform_joint" type="revolute">
+    <joint name="wrist_platform" type="revolute">
       <parent link="${prefix}bottom_parallel_link"/>
       <child link="${prefix}wrist_platform_link"/>
@@ -395,5 +395,5 @@
     </link>
     <!-- Joint 5: Wrist Pitch -->
-    <joint name="${prefix}wrist_pitch_joint" type="revolute">
+    <joint name="wrist_pitch" type="revolute">
       <parent link="${prefix}wrist_platform_link"/>
       <child link="${prefix}wrist_pitch_link"/>
@@ -425,5 +425,5 @@
     </link>
     <!-- Joint 6: Wrist Yaw-->
-    <joint name="${prefix}wrist_yaw_joint" type="revolute">
+    <joint name="wrist_yaw" type="revolute">
       <parent link="${prefix}wrist_pitch_link"/>
       <child link="${prefix}wrist_yaw_link"/>    <!--  defined from CAD file-->
@@ -454,5 +454,5 @@
     </link>
     <!-- Joint 7: Wrist Roll -->
-    <joint name="${prefix}wrist_roll_joint" type="revolute">
+    <joint name="wrist_roll" type="revolute">
       <parent link="${prefix}wrist_yaw_link"/>
       <child link="${prefix}wrist_roll_link"/>  <!-- -.039 & .055 defined from CAD file-->
@@ -486,5 +486,5 @@
     <transmission name="tran4">
       <type>transmission_interface/SimpleTransmission</type>
-      <joint name="${prefix}wrist_platform_joint"/>
+      <joint name="wrist_platform"/>
       <actuator name="motor4">
         <hardwareInterface>EffortJointInterface</hardwareInterface>
@@ -494,5 +494,5 @@
     <transmission name="tran5">
       <type>transmission_interface/SimpleTransmission</type>
-      <joint name="${prefix}wrist_pitch_joint"/>
+      <joint name="wrist_pitch"/>
       <actuator name="motor5">
         <hardwareInterface>EffortJointInterface</hardwareInterface>
@@ -502,5 +502,5 @@
     <transmission name="tran6">
       <type>transmission_interface/SimpleTransmission</type>
-      <joint name="${prefix}wrist_yaw_joint"/>
+      <joint name="wrist_yaw"/>
       <actuator name="motor6">
         <hardwareInterface>EffortJointInterface</hardwareInterface>
@@ -510,5 +510,5 @@
     <transmission name="tran7">
       <type>transmission_interface/SimpleTransmission</type>
-      <joint name="${prefix}wrist_roll_joint"/>
+      <joint name="wrist_roll"/>
       <actuator name="motor7">
         <hardwareInterface>EffortJointInterface</hardwareInterface>

File: dvrk_model/model/psm.base.urdf.xacro (robot description, xacro)
@@ -3,5 +3,5 @@
   <xacro:macro name="psm" params="prefix parent_link xyz rpy">
     <!-- fixed joint -->
-    <joint name="${prefix}fixed_joint" type="fixed">
+    <joint name="fixed" type="fixed">
       <parent link="${parent_link}"/>
       <child link="${prefix}psm_base_link"/>
@@ -18,5 +18,5 @@
     </link>
     <!-- joint 1 -->
-    <joint name="${prefix}outer_yaw_joint" type="revolute">
+    <joint name="outer_yaw" type="revolute">
       <parent link="${prefix}psm_base_link"/>
       <child link="${prefix}outer_yaw_link"/>
@@ -37,7 +37,7 @@
     <!-- Note: I can not put visual link here as it's parallel -->
     <!-- mechanism, so the outer_pitch_link does not have visual -->
-    <!-- link, all visual links mimic outer_pitch_joint value -->
+    <!-- link, all visual links mimic outer_pitch value -->
     <!-- joint 2: outer_pitch -->
-    <joint name="${prefix}outer_pitch_joint" type="revolute">
+    <joint name="outer_pitch" type="revolute">
       <parent link="${prefix}outer_yaw_link"/>
       <child link="${prefix}outer_pitch_link"/>
@@ -49,5 +49,5 @@
     <link name="${prefix}outer_pitch_link"/>
     <!-- joint 2-1: outer_pitch_1 -->
-    <joint name="${prefix}outer_pitch_joint_1" type="continuous">
+    <joint name="outer_pitch_1" type="continuous">
       <parent link="${prefix}outer_yaw_link"/>
       <child link="${prefix}outer_pitch_back_link"/>
@@ -55,5 +55,5 @@
       <!-- <origin rpy="-1.5708 -1.5708 0" xyz="0 0.0295 0.1495"/> -->
       <origin rpy="-1.5708 -1.5708 0" xyz="0 0.0295 0.5185"/>
-      <mimic joint="${prefix}outer_pitch_joint" multiplier="1"/>
+      <mimic joint="outer_pitch" multiplier="1"/>
     </joint>
     <!-- link 2-1: outer_pitch_back -->
@@ -67,10 +67,10 @@
     </link>
     <!-- joint 2-2: outer_pitch_2 -->
-    <joint name="${prefix}outer_pitch_joint_2" type="continuous">
+    <joint name="outer_pitch_2" type="continuous">
       <parent link="${prefix}outer_yaw_link"/>
       <child link="${prefix}outer_pitch_front_link"/>
       <axis xyz="0 0 1"/>
       <origin rpy="-1.5708 -1.5708 0" xyz="0 0.0295 0.4285"/>
-      <mimic joint="${prefix}outer_pitch_joint" multiplier="1"/>
+      <mimic joint="outer_pitch" multiplier="1"/>
     </joint>
     <!-- link 2-2: outer_pitch_front -->
@@ -84,10 +84,10 @@
     </link>
     <!-- joint 2-3: outer_pitch_3 -->
-    <joint name="${prefix}outer_pitch_joint_3" type="continuous">
+    <joint name="outer_pitch_3" type="continuous">
       <parent link="${prefix}outer_pitch_back_link"/>
       <child link="${prefix}outer_pitch_bottom_link"/>
       <axis xyz="0 0 1"/>
       <origin rpy="0 0 0" xyz="0.04178 0.15007 -0.0137"/>
-      <mimic joint="${prefix}outer_pitch_joint" multiplier="-1"/>
+      <mimic joint="outer_pitch" multiplier="-1"/>
     </joint>
     <!-- link 2-3: outer_pitch_bottom -->
@@ -101,10 +101,10 @@
     </link>
     <!-- joint 2-4: outer_pitch_4 -->
-    <joint name="${prefix}outer_pitch_joint_4" type="continuous">
+    <joint name="outer_pitch_4" type="continuous">
       <parent link="${prefix}outer_pitch_back_link"/>
       <child link="${prefix}outer_pitch_top_link"/>
       <axis xyz="0 0 1"/>
       <origin rpy="0 0 0" xyz="0.04209 0.18695 -0.02412"/>
-      <mimic joint="${prefix}outer_pitch_joint" multiplier="-1"/>
+      <mimic joint="outer_pitch" multiplier="-1"/>
     </joint>
     <!-- link 2-4: outer_pitch_top -->
@@ -118,10 +118,10 @@
     </link>
     <!-- joint 2-5: outer_pitch_5 -->
-    <joint name="${prefix}outer_pitch_joint_5" type="continuous">
+    <joint name="outer_pitch_5" type="continuous">
       <parent link="${prefix}outer_pitch_bottom_link"/>
       <child link="${prefix}outer_insertion_link"/>
       <axis xyz="0 0 1"/>
       <origin rpy="0 0 0" xyz="-0.520 0 -0.0155"/>
-      <mimic joint="${prefix}outer_pitch_joint" multiplier="1"/>
+      <mimic joint="outer_pitch" multiplier="1"/>
     </joint>
     <!-- link 2-5: outer_insertion -->
@@ -135,5 +135,5 @@
     </link>
     <!-- joint 3: insertion -->
-    <joint name="${prefix}outer_insertion_joint" type="prismatic">
+    <joint name="outer_insertion" type="prismatic">
       <!-- <parent link="${prefix}outer_insertion_link"/> -->
       <!-- <parent link="${prefix}psm_base_link"/> -->
@@ -154,5 +154,5 @@
     </link>
     <!-- joint 4: Outer Roll -->
-    <joint name="${prefix}outer_roll_joint" type="revolute">
+    <joint name="outer_roll" type="revolute">
       <parent link="${prefix}tool_main_link"/>
       <child link="${prefix}tool_wrist_link"/>
@@ -171,5 +171,5 @@
     </link>
     <!-- joint 4-1: outer roll shaft joint FIXED-->
-    <joint name="${prefix}outer_roll_shaft_joint" type="fixed">
+    <joint name="outer_roll_shaft" type="fixed">
       <parent link="${prefix}tool_wrist_link"/>
       <child link="${prefix}tool_wrist_shaft_link"/>

File: dvrk_model/model/psm.tool.caudier.urdf.xacro (robot description, xacro)
@@ -3,5 +3,5 @@
   <xacro:macro name="psm_tool_caudier" params="prefix">
     <!-- joint 5: Outer wrist pitch joint -->
-    <joint name="${prefix}outer_wrist_pitch_joint" type="revolute">
+    <joint name="outer_wrist_pitch" type="revolute">
       <parent link="${prefix}tool_wrist_shaft_link"/>
       <child link="${prefix}tool_wrist_caudier_link"/>
@@ -27,5 +27,5 @@
     </link>
     <!-- joint 6: Tool wrist yaw joint -->
-    <joint name="${prefix}outer_wrist_yaw_joint" type="revolute">
+    <joint name="outer_wrist_yaw" type="revolute">
       <parent link="${prefix}tool_wrist_caudier_link"/>
       <child link="${prefix}tool_wrist_caudier_link_shaft"/>
@@ -50,6 +50,23 @@
       </collision>
     </link>
-    <!-- joint 6-1: Outer open angle 1 -->
-    <joint name="${prefix}outer_wrist_open_angle_joint" type="revolute">
+    <!-- joint 7-0: Outer open angle 1  -->
+    <joint name="jaw" type="revolute">
+      <parent link="${prefix}tool_wrist_caudier_link_shaft"/>
+      <child link="${prefix}tool_wrist_caudier_ee_link_0"/>
+      <axis xyz="0 0 1"/>
+      <origin rpy="0 0 0" xyz="0 0 0"/>
+      <limit lower="0" upper="1.5707" velocity=".4" effort="1000"/>
+    </joint>
+    <!-- link 7-0: Outer open angle virtual -->
+    <link name="${prefix}tool_wrist_caudier_ee_link_0">
+      <visual>
+        <origin rpy="0 0 0" xyz="0 0 0"/>
+        <geometry>
+          <box size="0 0 0" />
+        </geometry>
+      </visual>
+    </link>
+    <!-- joint 7-1: Outer open angle 1 -->
+    <joint name="jaw_mimic_1" type="revolute">
       <parent link="${prefix}tool_wrist_caudier_link_shaft"/>
       <child link="${prefix}tool_wrist_caudier_link_2_left"/>
@@ -57,22 +74,17 @@
       <origin rpy="0 0 0" xyz="0 0 0"/>
       <limit lower="0" upper="1.5707" velocity=".4" effort="1000"/>
+      <mimic joint="jaw" multiplier="0.5"/>
     </joint>
-    <!-- link 6-1: Outer open angle link 1 -->
+    <!-- link 7-1: Outer open angle link 1 -->
     <link name="${prefix}tool_wrist_caudier_link_2_left">
       <visual>
         <origin rpy="0.0 0 0.0" xyz="0 0 0.00195"/>
         <geometry>
-          <mesh filename="package://dvrk_model/meshes/psm/tool_wrist_caudier_link_2_left.stl"/>
+          <mesh filename="package://dvrk_model/meshes/psm/tool_wrist_caudier_link_2.stl"/>
         </geometry>
       </visual>
-      <collision>
-        <origin rpy="0.0 0 0.0" xyz="0 0 0.00195"/>
-        <geometry>
-          <mesh filename="package://dvrk_model/meshes/psm/tool_wrist_caudier_link_2_left.stl"/>
-        </geometry>
-      </collision>
     </link>
-    <!-- joint 6-2: Outer open angle 2  -->
-    <joint name="${prefix}outer_wrist_open_angle_joint_mimic" type="revolute">
+    <!-- joint 7-2: Outer open angle 2  -->
+    <joint name="jaw_mimic_2" type="revolute">
       <parent link="${prefix}tool_wrist_caudier_link_shaft"/>
       <child link="${prefix}tool_wrist_caudier_link_2_right"/>
@@ -80,28 +92,20 @@
       <origin rpy="3.1415926 0 0" xyz="0 0 0"/>
       <limit lower="0" upper="1.5707" velocity=".4" effort="1000"/>
-      <mimic joint="${prefix}outer_wrist_open_angle_joint" multiplier="1"/>
+      <mimic joint="jaw" multiplier="0.5"/>
     </joint>
-    <!-- link 6-2: Outer open angle link 2 -->
+    <!-- link 7-2: Outer open angle link 2 -->
     <link name="${prefix}tool_wrist_caudier_link_2_right">
       <visual>
         <origin rpy="0 0 -3.1415926" xyz="0 0 0.00195"/>
         <geometry>
-          <mesh filename="package://dvrk_model/meshes/psm/tool_wrist_caudier_link_2_right.stl"/>
+          <mesh filename="package://dvrk_model/meshes/psm/tool_wrist_caudier_link_2.stl"/>
         </geometry>
       </visual>
-      <collision>
-        <origin rpy="0 0 -3.1415926" xyz="0 0 0.00195"/>
-        <geometry>
-          <mesh filename="package://dvrk_model/meshes/psm/tool_wrist_caudier_link_2_right.stl"/>
-        </geometry>
-      </collision>
     </link>
-    <!-- joint 6-3:   -->
-    <joint name="${prefix}tool_wrist_caudier_ee_joint" type="revolute">
+    <!-- tool tip   -->
+    <joint name="tool_wrist_caudier_ee" type="fixed">
       <parent link="${prefix}tool_wrist_caudier_link_shaft"/>
       <child link="${prefix}tool_wrist_caudier_ee_link"/>
-      <axis xyz="0 0 1"/>
       <origin rpy="0.0 1.5708 1.5708" xyz="0 0 0"/>
-      <limit lower="-1.5707" upper="1.5707" velocity=".4" effort="1000"/>
     </joint>
     <!-- link 6-3:  -->
