Commit message: dvrk_model: fixed ECM urdf xacro files to use new joint names and avoid python joint_publisher

File: dvrk_model/model/ECM.urdf.xacro (robot description, xacro)
@@ -1,208 +1,10 @@
 <?xml version="1.0" ?>
-<robot name="mtm" xmlns:xacro="http://www.ros.org/wiki/xacro">
-  <!-- Colors -->
-  <xacro:include filename="$(find dvrk_model)/model/common.urdf.xacro"/>
-  <!-- Macro for da Vinci Endoscope Camera Manipulator (ECM) -->
-  <xacro:macro name="ecm" params="prefix parent_link xyz rpy">
-    <!-- Joint 0: Fixed to World-->
-    <joint name="${prefix}_setup_fixed_joint" type="fixed">
-      <parent link="${parent_link}"/>
-      <child link="${prefix}_setup_base_link"/>
-      <origin rpy="${rpy}" xyz="${xyz}"/>
-    </joint>
-    <link name="${prefix}_setup_base_link"/>
-    <joint name="${prefix}_setup_tip_joint" type="fixed">
-      <parent link="${prefix}_setup_base_link"/>
-      <child link="${prefix}_setup_link"/>
-      <origin rpy="-0.87046370379 0 -${PI/2}" xyz="0.91324 -0.02111 0.03166"/>
-      <axis xyz="0 0 1"/>
-    </joint>
-    <link name="${prefix}_setup_link">
-      <visual>
-        <origin rpy="0 0 0" xyz="0 0 0"/>
-        <geometry>
-          <mesh filename="package://dvrk_model/meshes/ecm/Endo_Arm.STL"/>
-        </geometry>
-	<material name="DaVinciRed"/>
-      </visual>
-      <collision>
-        <origin rpy="0 0 0" xyz="0 0 0"/>
-        <geometry>
-          <mesh filename="package://dvrk_model/meshes/ecm/Endo_Arm.STL"/>
-        </geometry>
-      </collision>
-    </link>
-    <!-- Joint 0: Fixed to Setup Joint-->
-    <joint name="${prefix}_fixed_joint" type="fixed">
-      <parent link="${prefix}_setup_link"/>
-      <child link="${prefix}_base_link"/>
-      <origin rpy="0 0 0" xyz="0 0.603 0"/>
-    </joint>
-    <link name="${prefix}_base_link"/>
-    <!-- Joint 1: Outer Yaw -->
-    <joint name="${prefix}_yaw_joint" type="revolute">
-      <parent link="${prefix}_base_link"/>
-      <child link="${prefix}_yaw_link"/>
-      <origin rpy="0 -${PI/2} ${PI/2}" xyz="0 0 0"/>
-      <axis xyz="0 0 1"/>
-      <!--rotates about z axis-->
-      <!--limit effort and velocity picked arbitrarily check-->
-      <limit effort="50.0" lower="${-75/180*PI}" upper="${PI/4}" velocity="2"/>
-      <joint_properties damping="1.0" friction="0.0"/>
-    </joint>
-    <link name="${prefix}_yaw_link">
-      <visual>
-        <origin rpy="0 0 -${PI/2}" xyz="0.0 0 0.603"/>
-        <geometry>
-          <mesh filename="package://dvrk_model/meshes/ecm/Endo_Link_5.STL"/>
-        </geometry>
-	<material name="DaVinciGreen"/>
-      </visual>
-      <collision>
-        <origin rpy="0 0 -${PI/2}" xyz="0.0 0 0.603"/>
-        <geometry>
-          <mesh filename="package://dvrk_model/meshes/ecm/Endo_Link_5.STL"/>
-        </geometry>
-      </collision>
-    </link>
-    <!-- Joint 2: Pitch -->
-    <joint name="${prefix}_pitch_joint" type="revolute">
-      <parent link="${prefix}_yaw_link"/>
-      <child link="${prefix}_pitch_link"/>
-      <origin rpy="-${PI/2} -${PI/2} 0" xyz="0 0 0"/>
-      <axis xyz="0 0 1"/>
-      <limit effort="100.0" lower="${-PI/4}" upper="${PI*65/180}" velocity="10"/>
-      <joint_properties damping="1.0" friction="0.0"/>
-    </joint>
-    <link name="${prefix}_pitch_link"/>
-    <joint name="${prefix}_pitch_joint_0" type="continuous">
-      <parent link="${prefix}_yaw_link"/>
-      <child link="${prefix}_pitch_link_1"/>
-      <origin rpy="-${PI/2} -${PI/2} 0" xyz="0 0 0.378"/>
-      <axis xyz="0 0 1"/>
-      <joint_properties damping="1.0" friction="0.0"/>
-      <mimic joint="${prefix}_pitch_joint" multiplier="1"/>
-    </joint>
-    <link name="${prefix}_pitch_link_1">
-      <visual>
-        <origin rpy="${PI} 0 ${PI*78.5/180}" xyz="0.0 0 0.0"/>
-        <geometry>
-          <mesh filename="package://dvrk_model/meshes/ecm/Endo_Link_5_2.STL"/>
-        </geometry>
-	<material name="DaVinciMedGray"/>
-      </visual>
-      <collision>
-        <origin rpy="${PI} 0 ${PI*78.5/180}" xyz="0.0 0 0.0"/>
-        <geometry>
-          <mesh filename="package://dvrk_model/meshes/ecm/Endo_Link_5_2.STL"/>
-        </geometry>
-      </collision>
-      <inertial>
-        <mass value=".9"/>
-        <inertia ixx="9.0" ixy="0.0" ixz="0.0" iyy="9.0" iyz="0.0" izz="9.0"/>
-      </inertial>
-    </link>
-    <joint name="${prefix}_pitch_joint_1" type="continuous">
-      <parent link="${prefix}_pitch_link_1"/>
-      <child link="${prefix}_pitch_link_2"/>
-      <origin rpy="0 0 0" xyz="0.0558629 0.274575 0"/>
-      <axis xyz="0 0 1"/>
-      <joint_properties damping="1.0" friction="0.0"/>
-      <mimic joint="${prefix}_pitch_joint" multiplier="-1"/>
-    </joint>
-    <link name="${prefix}_pitch_link_2">
-      <visual>
-        <origin rpy="0 0 0" xyz="0.0 0 -0.0225"/>
-        <geometry>
-          <mesh filename="package://dvrk_model/meshes/ecm/Endo_Link_6_2.STL"/>
-        </geometry>
-	<material name="DaVinciMedGray"/>
-      </visual>
-      <collision>
-        <origin rpy="0 0 0" xyz="0.0 0 -0.0225"/>
-        <geometry>
-          <mesh filename="package://dvrk_model/meshes/ecm/Endo_Link_6_2.STL"/>
-        </geometry>
-      </collision>
-      <inertial>
-        <mass value=".9"/>
-        <inertia ixx="9.0" ixy="0.0" ixz="0.0" iyy="9.0" iyz="0.0" izz="9.0"/>
-      </inertial>
-    </link>
-    <joint name="${prefix}_pitch_joint_2" type="continuous">
-      <parent link="${prefix}_pitch_link_2"/>
-      <child link="${prefix}_pitch_link_3"/>
-      <origin rpy="0 0 0" xyz="-0.340 0 0"/>
-      <axis xyz="0 0 1"/>
-      <joint_properties damping="1.0" friction="0.0"/>
-      <mimic joint="${prefix}_pitch_joint" multiplier="1"/>
-    </joint>
-    <link name="${prefix}_pitch_link_3">
-      <visual>
-        <origin rpy="0 0 -${PI/2}" xyz="0.0 0 0.025"/>
-        <geometry>
-          <mesh filename="package://dvrk_model/meshes/ecm/Endo_Link_7.STL"/>
-        </geometry>
-	<material name="DaVinciMedGray"/>
-      </visual>
-      <collision>
-        <origin rpy="0 0 -${PI/2}" xyz="0.0 0 0.025"/>
-        <geometry>
-          <mesh filename="package://dvrk_model/meshes/ecm/Endo_Link_7.STL"/>
-        </geometry>
-      </collision>
-      <inertial>
-        <mass value=".9"/>
-        <inertia ixx="9.0" ixy="0.0" ixz="0.0" iyy="9.0" iyz="0.0" izz="9.0"/>
-      </inertial>
-    </link>
-    <!-- Joint 3: Insertion -->
-    <joint name="${prefix}_insertion_joint" type="prismatic">
-      <parent link="${prefix}_pitch_link"/>
-      <child link="${prefix}_insertion_link"/>
-      <origin rpy="${PI/2} 0 0" xyz="0 0.3822 0"/>
-      <axis xyz="0 0 1"/>
-      <joint_properties damping="1.0" friction="0.0"/>
-      <limit effort="100.0" lower="0" upper="0.235" velocity="10"/>
-    </joint>
-    <link name="${prefix}_insertion_link">
-      <visual>
-        <origin rpy="0 0 -${PI/2}" xyz="0.0 0 -0.015"/>
-        <geometry>
-          <mesh filename="package://dvrk_model/meshes/ecm/Endo_Link_8.STL"/>
-        </geometry>
-	<material name="DaVinciBlue"/>
-      </visual>
-      <collision>
-        <origin rpy="0 0 -${PI/2}" xyz="0.0 0 -0.015"/>
-        <geometry>
-          <mesh filename="package://dvrk_model/meshes/ecm/Endo_Link_8.STL"/>
-        </geometry>
-      </collision>
-    </link>
-    <!-- Joint 4: Roll -->
-    <joint name="${prefix}_roll_joint" type="revolute">
-      <parent link="${prefix}_insertion_link"/>
-      <child link="${prefix}_roll_link"/>
-      <origin rpy="0 0 0" xyz="0 0 0.3829"/>
-      <axis xyz="0 0 1"/>
-      <joint_properties damping="1.0" friction="0.0"/>
-      <limit effort="100.0" lower="-${PI/2}" upper="${PI/2}" velocity="10"/>
-    </joint>
-    <link name="${prefix}_roll_link">
-      <visual>
-        <origin rpy="0 0 ${PI/2}" xyz="0.0 0 -0.3979"/>
-        <geometry>
-          <mesh filename="package://dvrk_model/meshes/ecm/EndoScope.STL"/>
-        </geometry>
-	<material name="DaVinciBlue"/>
-      </visual>
-      <collision>
-        <origin rpy="0 0 ${PI/2}" xyz="0.0 0 -0.3979"/>
-        <geometry>
-          <mesh filename="package://dvrk_model/meshes/ecm/EndoScope.STL"/>
-        </geometry>
-      </collision>
-    </link>
-  </xacro:macro>
+<robot name="ecm" xmlns:xacro="http://www.ros.org/wiki/xacro">
+  <!-- Macros -->
+  <xacro:include filename="$(find dvrk_model)/model/ecm.urdf.xacro"/>
+  <link name="world"/>
+  <xacro:ecm
+      prefix="ecm"
+      parent_link="world"
+      xyz="0 0.0 0.0" rpy="0.0 0.0 0.0"/>
 </robot>
