Commit message: fixed psm xacro file

File: dvrk_model/model/psm.urdf.xacro (robot description, xacro)
@@ -2,18 +2,4 @@
 <robot name="dvrk_psm" xmlns:xacro="http://www.ros.org/wiki/xacro">
   <xacro:macro name="psm" params="prefix parent_link xyz rpy">
-    <!-- fixed joint -->
-    <!-- <joint name="${prefix}fixed_joint" type="fixed"> -->
-    <!--   <parent link="${parent_link}"/> -->
-    <!--   <child link="${prefix}remote_center_link"/> -->
-    <!--   <origin rpy="${rpy}" xyz="${xyz}"/> -->
-    <!-- </joint> -->
-    <!-- link rc: remote centre link -->
-    <!-- <link name="${prefix}remote_center_link" />    -->
-    <!-- fixed joint -->
-    <!-- <joint name="${prefix}rc_fixed_joint" type="fixed"> -->
-    <!--   <parent link="${prefix}remote_center_link"/> -->
-    <!--   <child link="${prefix}psm_base_link"/> -->
-    <!--   <origin rpy="0 0 0" xyz="0 0 0"/> -->
-    <!-- </joint> -->
     <!-- fixed joint -->
     <joint name="${prefix}fixed_joint" type="fixed">
@@ -151,9 +137,9 @@
     <joint name="${prefix}outer_insertion_joint" type="prismatic">
       <!-- <parent link="${prefix}outer_insertion_link"/> -->
-      <parent link="${prefix}psm_base_link"/>
+      <!-- <parent link="${prefix}psm_base_link"/> -->
+      <parent link="${prefix}outer_pitch_link"/>
       <child link="${prefix}tool_main_link"/>
       <axis xyz="0 0 1"/>
-      <!-- <origin rpy="1.5708 0 0" xyz="-0.0403 0.23622 0"/> -->
-      <origin rpy="0 3.1415926 1.5708" xyz="0 0 0"/>
+      <origin rpy="1.5708 0 0" xyz="0 0.4318 0"/>
       <limit lower="0" upper="0.240" velocity=".4" effort="1000"/>
     </joint>
@@ -161,5 +147,5 @@
     <link name="${prefix}tool_main_link">
       <visual>
-        <!-- <origin rpy="0 0 1.5708" xyz="0 0 0"/> -->
+        <origin rpy="0 0 1.5708" xyz="0 0 0.041"/>
         <geometry>
           <mesh filename="package://dvrk_model/meshes/psm/tool_main.dae"/>
@@ -167,15 +153,13 @@
       </visual>
     </link>
-    <!-- joint 4-1: Outer Roll -->
+    <!-- joint 4: Outer Roll -->
     <joint name="${prefix}outer_roll_joint" type="revolute">
       <parent link="${prefix}tool_main_link"/>
       <child link="${prefix}tool_wrist_link"/>
       <axis xyz="0 0 1"/>
-      <!-- 0.36680 + 0.0091 = 0.3759 -->
-      <!-- <origin rpy="0 0 0" xyz="0 0 0.3759"/> -->
       <origin rpy="0 0 0" xyz="0 0 0.4162"/>
       <limit lower="-2.2689" upper="2.2689" velocity=".4" effort="1000"/>
     </joint>
-    <!-- link 4-1: tool_main_link -->
+    <!-- link 4: tool_wrist_link -->
     <link name="${prefix}tool_wrist_link">
       <visual>
@@ -186,4 +170,5 @@
       </visual>
     </link>
+    <!-- joint 4-1: outer roll shaft joint FIXED-->
     <joint name="${prefix}outer_roll_shaft_joint" type="fixed">
       <parent link="${prefix}tool_wrist_link"/>
@@ -192,4 +177,5 @@
       <origin rpy="0 0 0" xyz="0 0 0.0"/>
     </joint>
+    <!-- link 4-1: tool_wrist_shaft_link -->
     <link name="${prefix}tool_wrist_shaft_link">
       <visual>

Commit message: major renaming and refactoring of psm xacro files

File: dvrk_model/model/psm.urdf.xacro (robot description, xacro)
@@ -1,260 +1,25 @@
-<?xml version="1.0" encoding="utf-8"?>
+<?xml version="1.0" ?>
 <robot name="dvrk_psm" xmlns:xacro="http://www.ros.org/wiki/xacro">
-  <xacro:macro name="psm" params="prefix parent_link xyz rpy">
-    <!-- fixed joint -->
-    <joint name="${prefix}fixed_joint" type="fixed">
-      <parent link="${parent_link}"/>
-      <child link="${prefix}psm_base_link"/>
-      <origin rpy="${rpy}" xyz="${xyz}"/>
-    </joint>
-    <!-- link 0: psm base link -->
-    <link name="${prefix}psm_base_link">
-      <visual>
-        <origin rpy="1.5708 0 3.1416" xyz="0.039 -0.40788 -0.07879"/>
-        <geometry>
-          <mesh filename="package://dvrk_model/meshes/psm/psm_base.dae"/>
-        </geometry>
-      </visual>
-    </link>
-    <!-- joint 1 -->
-    <joint name="${prefix}outer_yaw_joint" type="revolute">
-      <parent link="${prefix}psm_base_link"/>
-      <child link="${prefix}outer_yaw_link"/>
-      <axis xyz="0 0 1"/>
-      <!-- <origin rpy="1.5708 -1.5708 0" xyz="0.0 -0.369 0.0"/> -->
-      <origin rpy="0 -1.5708 1.5708" xyz="0.0 0.0 0.0"/>
-      <limit lower="-1.5707" upper="1.5707" velocity=".4" effort="1000"/>
-    </joint>
-    <!-- link 1: outer_yaw -->
-    <link name="${prefix}outer_yaw_link">
-      <visual>        <!-- <origin rpy="0 0 -1.5708" xyz="0.0125 0 0.1575"/> -->
-        <origin rpy="3.1416 0 1.5708" xyz="0.0125 0 0.5265"/>
-        <geometry>
-          <mesh filename="package://dvrk_model/meshes/psm/outer_yaw.dae"/>
-        </geometry>
-      </visual>
-    </link>
-    <!-- Note: I can not put visual link here as it's parallel -->
-    <!-- mechanism, so the outer_pitch_link does not have visual -->
-    <!-- link, all visual links mimic outer_pitch_joint value -->
-    <!-- joint 2: outer_pitch -->
-    <joint name="${prefix}outer_pitch_joint" type="revolute">
-      <parent link="${prefix}outer_yaw_link"/>
-      <child link="${prefix}outer_pitch_link"/>
-      <axis xyz="0 0 1"/>
-      <origin rpy="-1.5708 -1.5708 0" xyz="0 0 0"/>
-      <limit lower="-0.7854" upper="0.7854" velocity=".4" effort="1000"/>
-    </joint>
-    <!-- link 2: outer_pitch_link -->
-    <link name="${prefix}outer_pitch_link"/>
-    <!-- joint 2-1: outer_pitch_1 -->
-    <joint name="${prefix}outer_pitch_joint_1" type="continuous">
-      <parent link="${prefix}outer_yaw_link"/>
-      <child link="${prefix}outer_pitch_back_link"/>
-      <axis xyz="0 0 1"/>
-      <!-- <origin rpy="-1.5708 -1.5708 0" xyz="0 0.0295 0.1495"/> -->
-      <origin rpy="-1.5708 -1.5708 0" xyz="0 0.0295 0.5185"/>
-      <mimic joint="${prefix}outer_pitch_joint" multiplier="1"/>
-    </joint>
-    <!-- link 2-1: outer_pitch_back -->
-    <link name="${prefix}outer_pitch_back_link">
-      <visual>
-        <origin rpy="0 0 -0.27129" xyz="0 0 0"/>
-        <geometry>
-          <mesh filename="package://dvrk_model/meshes/psm/outer_pitch_back.dae"/>
-        </geometry>
-      </visual>
-    </link>
-    <!-- joint 2-2: outer_pitch_2 -->
-    <joint name="${prefix}outer_pitch_joint_2" type="continuous">
-      <parent link="${prefix}outer_yaw_link"/>
-      <child link="${prefix}outer_pitch_front_link"/>
-      <axis xyz="0 0 1"/>
-      <origin rpy="-1.5708 -1.5708 0" xyz="0 0.0295 0.4285"/>
-      <mimic joint="${prefix}outer_pitch_joint" multiplier="1"/>
-    </joint>
-    <!-- link 2-2: outer_pitch_front -->
-    <link name="${prefix}outer_pitch_front_link">
-      <visual>
-        <origin rpy="0 0 -0.27129" xyz="0 0 0"/>
-        <geometry>
-          <mesh filename="package://dvrk_model/meshes/psm/outer_pitch_front.dae"/>
-        </geometry>
-      </visual>
-    </link>
-    <!-- joint 2-3: outer_pitch_3 -->
-    <joint name="${prefix}outer_pitch_joint_3" type="continuous">
-      <parent link="${prefix}outer_pitch_back_link"/>
-      <child link="${prefix}outer_pitch_bottom_link"/>
-      <axis xyz="0 0 1"/>
-      <origin rpy="0 0 0" xyz="0.04178 0.15007 -0.0137"/>
-      <mimic joint="${prefix}outer_pitch_joint" multiplier="-1"/>
-    </joint>
-    <!-- link 2-3: outer_pitch_bottom -->
-    <link name="${prefix}outer_pitch_bottom_link">
-      <visual>
-        <origin rpy="0 -1.5708 0" xyz="0.009 0 0"/>
-        <geometry>
-          <mesh filename="package://dvrk_model/meshes/psm/outer_pitch_bottom.dae"/>
-        </geometry>
-      </visual>
-    </link>
-    <!-- joint 2-4: outer_pitch_4 -->
-    <joint name="${prefix}outer_pitch_joint_4" type="continuous">
-      <parent link="${prefix}outer_pitch_back_link"/>
-      <child link="${prefix}outer_pitch_top_link"/>
-      <axis xyz="0 0 1"/>
-      <origin rpy="0 0 0" xyz="0.04209 0.18695 -0.02412"/>
-      <mimic joint="${prefix}outer_pitch_joint" multiplier="-1"/>
-    </joint>
-    <!-- link 2-4: outer_pitch_top -->
-    <link name="${prefix}outer_pitch_top_link">
-      <visual>
-        <origin rpy="0 -1.5708 0" xyz="0.009 0 0"/>
-        <geometry>
-          <mesh filename="package://dvrk_model/meshes/psm/outer_pitch_top.dae"/>
-        </geometry>
-      </visual>
-    </link>
-    <!-- joint 2-5: outer_pitch_5 -->
-    <joint name="${prefix}outer_pitch_joint_5" type="continuous">
-      <parent link="${prefix}outer_pitch_bottom_link"/>
-      <child link="${prefix}outer_insertion_link"/>
-      <axis xyz="0 0 1"/>
-      <origin rpy="0 0 0" xyz="-0.520 0 -0.0155"/>
-      <mimic joint="${prefix}outer_pitch_joint" multiplier="1"/>
-    </joint>
-    <!-- link 2-5: outer_insertion -->
-    <link name="${prefix}outer_insertion_link">
-      <visual>
-        <origin rpy="0 -1.5708 1.5708" xyz="0.02528 0.429 0"/>
-        <geometry>
-          <mesh filename="package://dvrk_model/meshes/psm/outer_insertion.dae"/>
-        </geometry>
-      </visual>
-    </link>
-    <!-- joint 3: insertion -->
-    <joint name="${prefix}outer_insertion_joint" type="prismatic">
-      <!-- <parent link="${prefix}outer_insertion_link"/> -->
-      <!-- <parent link="${prefix}psm_base_link"/> -->
-      <parent link="${prefix}outer_pitch_link"/>
-      <child link="${prefix}tool_main_link"/>
-      <axis xyz="0 0 1"/>
-      <origin rpy="1.5708 0 0" xyz="0 0.4318 0"/>
-      <limit lower="0" upper="0.240" velocity=".4" effort="1000"/>
-    </joint>
-    <!-- link 3: tool_main_link -->
-    <link name="${prefix}tool_main_link">
-      <visual>
-        <origin rpy="0 0 1.5708" xyz="0 0 0.041"/>
-        <geometry>
-          <mesh filename="package://dvrk_model/meshes/psm/tool_main.dae"/>
-        </geometry>
-      </visual>
-    </link>
-    <!-- joint 4: Outer Roll -->
-    <joint name="${prefix}outer_roll_joint" type="revolute">
-      <parent link="${prefix}tool_main_link"/>
-      <child link="${prefix}tool_wrist_link"/>
-      <axis xyz="0 0 1"/>
-      <origin rpy="0 0 0" xyz="0 0 0.4162"/>
-      <limit lower="-2.2689" upper="2.2689" velocity=".4" effort="1000"/>
-    </joint>
-    <!-- link 4: tool_wrist_link -->
-    <link name="${prefix}tool_wrist_link">
-      <visual>
-        <origin rpy="0 0 1.5708" xyz="0 0 -0.0091"/>
-        <geometry>
-          <mesh filename="package://dvrk_model/meshes/psm/tool_wrist_link.dae"/>
-        </geometry>
-      </visual>
-    </link>
-    <!-- joint 4-1: outer roll shaft joint FIXED-->
-    <joint name="${prefix}outer_roll_shaft_joint" type="fixed">
-      <parent link="${prefix}tool_wrist_link"/>
-      <child link="${prefix}tool_wrist_shaft_link"/>
-      <axis xyz="0 0 1"/>
-      <origin rpy="0 0 0" xyz="0 0 0.0"/>
-    </joint>
-    <!-- link 4-1: tool_wrist_shaft_link -->
-    <link name="${prefix}tool_wrist_shaft_link">
-      <visual>
-        <origin rpy="1.5708 0 0" xyz="0 0.00401 0"/>
-        <geometry>
-          <mesh filename="package://dvrk_model/meshes/psm/tool_wrist_shaft_link.dae"/>
-        </geometry>
-      </visual>
-    </link>
-    <!-- joint 5: Outer wrist pitch joint -->
-    <joint name="${prefix}outer_wrist_pitch_joint" type="revolute">
-      <parent link="${prefix}tool_wrist_shaft_link"/>
-      <child link="${prefix}tool_wrist_sca_link"/>
-      <axis xyz="0 0 1"/>
-      <origin rpy="-1.5708 -1.5708 0" xyz="0 0 0"/>
-      <limit lower="-1.5707" upper="1.5707" velocity=".4" effort="1000"/>
-    </joint>
-    <!-- link 5: tool_wrist_sca_link -->
-    <link name="${prefix}tool_wrist_sca_link">
-      <visual>
-        <!-- <origin rpy="0 3.1416 0" xyz="0 0 0"/> -->
-        <origin rpy="1.5708 3.1416 0" xyz="0.0051 0.0032 0"/>
-        <geometry>
-          <mesh filename="package://dvrk_model/meshes/psm/tool_wrist_sca_link.dae"/>
-        </geometry>
-      </visual>
-    </link>
-    <!-- joint 6: Outer wrist yaw joint -->
-    <joint name="${prefix}outer_wrist_yaw_joint" type="revolute">
-      <parent link="${prefix}tool_wrist_sca_link"/>
-      <child link="${prefix}tool_wrist_sca_shaft_link"/>
-      <axis xyz="0 0 1"/>
-      <origin rpy="-1.5708 -1.5708 0" xyz="0.0091 0 0"/>
-      <!-- +/- 80 deg -->
-      <limit lower="-1.3963" upper="1.3963" velocity=".4" effort="1000"/>
-    </joint>
-    <!-- link 6: tool_wrist_sca_shaft_link -->
-    <link name="${prefix}tool_wrist_sca_shaft_link">
-      <visual>
-        <origin rpy="0 0 0" xyz="0 -0.0002 -0.0025"/>
-        <geometry>
-          <mesh filename="package://dvrk_model/meshes/psm/tool_wrist_sca_shaft_link.dae"/>
-        </geometry>
-      </visual>
-    </link>
-    <!-- joint 7-1: Outer open angle 1  -->
-    <joint name="${prefix}outer_wrist_open_angle_joint_1" type="revolute">
-      <parent link="${prefix}tool_wrist_sca_shaft_link"/>
-      <child link="${prefix}tool_wrist_sca_ee_link_1"/>
-      <axis xyz="0 0 1"/>
-      <origin rpy="0 0 0" xyz="0 0 0"/>
-      <limit lower="0" upper="1.5707" velocity=".4" effort="1000"/>
-    </joint>
-    <!-- link 7-1: Outer open angle link 1 -->
-    <link name="${prefix}tool_wrist_sca_ee_link_1">
-      <visual>
-        <origin rpy="0 0 0" xyz="0 0 0"/>
-        <geometry>
-          <mesh filename="package://dvrk_model/meshes/psm/tool_wrist_sca_link_2.dae"/>
-        </geometry>
-      </visual>
-    </link>
-    <!-- joint 7-2: Outer open angle 2   -->
-    <joint name="${prefix}outer_wrist_open_angle_joint_2" type="revolute">
-      <parent link="${prefix}tool_wrist_sca_shaft_link"/>
-      <child link="${prefix}tool_wrist_sca_ee_link_2"/>
-      <axis xyz="0 0 1"/>
-      <origin rpy="0 0 0" xyz="0 0 0"/>
-      <limit lower="-1.5707" upper="1.5707" velocity=".4" effort="1000"/>
-      <mimic joint="${prefix}outer_wrist_open_angle_joint_1" multiplier="-1"/>
-    </joint>
-    <!-- link 7-2: Outer open angle link 2 -->
-    <link name="${prefix}tool_wrist_sca_ee_link_2">
-      <visual>
-        <origin rpy="0 3.1516 0" xyz="0 0 0"/>
-        <geometry>
-          <mesh filename="package://dvrk_model/meshes/psm/tool_wrist_sca_link_2.dae"/>
-        </geometry>
-      </visual>
-    </link>
+  <!-- Macros -->
+  <xacro:include filename="$(find dvrk_model)/model/psm.base.urdf.xacro"/>
+  <xacro:include filename="$(find dvrk_model)/model/psm.tool.sca.urdf.xacro"/>
+  <xacro:include filename="$(find dvrk_model)/model/psm.tool.caudier.urdf.xacro"/>
+  <!-- Macro for psm with sca -->
+  <xacro:macro name="psm_sca" params="prefix parent_link xyz rpy">
+    <xacro:psm
+        prefix="${prefix}"
+        parent_link="${parent_link}"
+        xyz="${xyz}" rpy="${rpy}"/>
+    <xacro:psm_tool_sca
+        prefix="${prefix}"/>
+  </xacro:macro>
+  <!-- Macro for psm with caudier -->
+  <xacro:macro name="psm_caudier" params="prefix parent_link xyz rpy">
+    <xacro:psm
+        prefix="${prefix}"
+        parent_link="${parent_link}"
+        xyz="${xyz}" rpy="${rpy}"/>
+    <xacro:psm_tool_caudier
+        prefix="${prefix}"/>
   </xacro:macro>
 </robot>

File: dvrk_model/model/psm_one.urdf.xacro (robot description, xacro)
@@ -4,5 +4,5 @@
   <xacro:include filename="$(find dvrk_model)/model/psm.urdf.xacro"/>
   <link name="world"/>
-  <xacro:psm
+  <xacro:psm_sca
       prefix="one_"
       parent_link="world"

File: dvrk_model/model/psm_two.urdf.xacro (robot description, xacro)
@@ -4,5 +4,5 @@
   <xacro:include filename="$(find dvrk_model)/model/psm.urdf.xacro"/>
   <link name="world"/>
-  <xacro:psm
+  <xacro:psm_caudier
       prefix="two_"
       parent_link="world"

Commit message: Adding snake tool

File: dvrk_model/model/psm.urdf.xacro (robot description, xacro)
@@ -5,4 +5,14 @@
   <xacro:include filename="$(find dvrk_model)/model/psm.tool.sca.urdf.xacro"/>
   <xacro:include filename="$(find dvrk_model)/model/psm.tool.caudier.urdf.xacro"/>
+  <xacro:include filename="$(find dvrk_model)/model/psm.tool.snake.urdf.xacro"/>
+  <!-- Macro for psm with snake -->
+  <xacro:macro name="psm_snake" params="prefix parent_link xyz rpy">
+    <xacro:psm
+        prefix="${prefix}"
+        parent_link="${parent_link}"
+        xyz="${xyz}" rpy="${rpy}"/>
+    <xacro:psm_tool_snake
+        prefix="${prefix}"/>
+  </xacro:macro>
   <!-- Macro for psm with sca -->
   <xacro:macro name="psm_sca" params="prefix parent_link xyz rpy">
