Commit message: Updated snake urdf file

File: dvrk_model/model/psm.tool.snake.urdf.xacro (robot description, xacro)
@@ -3,27 +3,10 @@
   <!-- sca  -->
   <xacro:macro name="psm_tool_snake" params="prefix">
-    <!-- joint 5: Outer wrist pitch1 joint -->
+    <!-- joint 6: Outer wrist pitch1 joint -->
     <joint name="outer_wrist_pitch1" type="revolute">
       <parent link="${prefix}tool_wrist_shaft_link"/>
-      <child link="${prefix}tool_snake_base_link"/>
-      <axis xyz="0 0 1"/>
-      <origin rpy="-1.5707 -1.5708 0" xyz="0 0 0.0"/>
-      <limit lower="-1.5707" upper="1.5707" velocity=".4" effort="1000"/>
-    </joint>
-    <!-- link 5: tool_snake_base_link -->
-    <link name="${prefix}tool_snake_base_link">
-      <visual>
-        <origin rpy="0 1.5708 0" xyz="0 0 0"/>
-        <geometry>
-          <mesh filename="package://dvrk_model/meshes/psm/snake_tool/link_0.STL"/>
-        </geometry>
-      </visual>
-    </link>
-    <!-- joint 6: Outer wrist yaw1 joint -->
-    <joint name="outer_wrist_yaw1" type="revolute">
-      <parent link="${prefix}tool_snake_base_link"/>
       <child link="${prefix}tool_snake_disc1_link"/>
       <axis xyz="0 0 1"/>
-      <origin rpy="-1.5708 0 0" xyz="0.0034 0 0"/>
+      <origin rpy="-1.5708 -1.5708 0" xyz="0.0 0 0"/>
       <limit lower="-1.3963" upper="1.3963" velocity=".4" effort="1000"/>
     </joint>
@@ -31,5 +14,5 @@
     <link name="${prefix}tool_snake_disc1_link">
       <visual>
-        <origin rpy="0 0 0" xyz="-0.0034 0 0"/>
+        <origin rpy="1.5708 0 0" xyz="0.0027 0 0"/>
         <geometry>
           <mesh filename="package://dvrk_model/meshes/psm/snake_tool/link_1.STL"/>
@@ -37,10 +20,10 @@
       </visual>
     </link>
-   <!-- joint 7: Outer wrist yaw2 joint -->
-    <joint name="outer_wrist_yaw2" type="revolute">
+    <!-- joint 7: Outer wrist yaw1 joint -->
+    <joint name="outer_wrist_yaw1" type="revolute">
       <parent link="${prefix}tool_snake_disc1_link"/>
       <child link="${prefix}tool_snake_disc2_link"/>
       <axis xyz="0 0 1"/>
-      <origin rpy="0 0 0" xyz="0.0034 0 0"/>
+      <origin rpy="-1.5708 0 0" xyz="0.0034 0 0"/>
       <limit lower="-1.3963" upper="1.3963" velocity=".4" effort="1000"/>
     </joint>
@@ -48,5 +31,5 @@
     <link name="${prefix}tool_snake_disc2_link">
       <visual>
-        <origin rpy="-1.5708 0 0" xyz="-0.0034 0 0"/>
+        <origin rpy="1.5708 0 0" xyz="0.0027 0 0"/>
         <geometry>
           <mesh filename="package://dvrk_model/meshes/psm/snake_tool/link_2.STL"/>
@@ -54,10 +37,10 @@
       </visual>
     </link>
-    <!-- joint 8: Outer wrist pitch2 joint -->
-    <joint name="outer_wrist_pitch2" type="revolute">
+    <!-- joint 8: Outer wrist yaw2 joint -->
+    <joint name="outer_wrist_yaw2" type="revolute">
       <parent link="${prefix}tool_snake_disc2_link"/>
       <child link="${prefix}tool_snake_disc3_link"/>
       <axis xyz="0 0 1"/>
-      <origin rpy="1.5708 -1.5708 0" xyz="0.0034 0 0"/>
+      <origin rpy="0 0 0" xyz="0.0034 0 0"/>
       <limit lower="-1.3963" upper="1.3963" velocity=".4" effort="1000"/>
     </joint>
@@ -65,5 +48,5 @@
     <link name="${prefix}tool_snake_disc3_link">
       <visual>
-        <origin rpy="0 0 -1.5708" xyz="0 0.0034 0"/>
+        <origin rpy="1.5708 0 0" xyz="0.0027 0 0"/>
         <geometry>
           <mesh filename="package://dvrk_model/meshes/psm/snake_tool/link_3.STL"/>
@@ -71,42 +54,25 @@
       </visual>
     </link>
-  <!-- Fixed Gripper Holder joints -->
-    <!-- fixed Joint 0 -->
-    <joint name="outer_wrist_jaw_fixed1" type="revolute">
+    <!-- joint 9: Outer wrist pitch2 joint -->
+    <joint name="outer_wrist_pitch2" type="revolute">
       <parent link="${prefix}tool_snake_disc3_link"/>
-      <child link="${prefix}tool_snake_jaw_fixed1_link"/>
+      <child link="${prefix}tool_snake_end_link"/>
       <axis xyz="0 0 1"/>
-      <origin rpy="0 0 0" xyz="0 0 0.0"/>
+      <origin rpy="1.5708 -1.5708 0" xyz="0.0034 0 0"/>
       <limit lower="-1.3963" upper="1.3963" velocity=".4" effort="1000"/>
     </joint>
-    <!-- link 9F-0: tool_snake_jaw_fixed1_link -->
-    <link name="${prefix}tool_snake_jaw_fixed1_link">
+    <!-- link 9: tool_snake_end_link -->
+    <link name="${prefix}tool_snake_end_link">
       <visual>
-        <origin rpy="-1.5708 0 0" xyz="0 -0.0061 0"/>
+        <origin rpy="0 1.5708 0" xyz="0 -0.0027 0"/>
         <geometry>
-          <mesh filename="package://dvrk_model/meshes/psm/snake_tool/gripper_0.STL"/>
-        </geometry>
-      </visual>
-    </link>
-    <!-- fixed Joint 1 -->
-    <joint name="outer_wrist_jaw_fixed2" type="fixed">
-      <parent link="${prefix}tool_snake_jaw_fixed1_link"/>
-      <child link="${prefix}tool_snake_jaw_fixed2_link"/>
-      <axis xyz="0 0 1"/>
-      <origin rpy="0 0 0" xyz="0 0 0.0"/>
-    </joint>
-    <!-- link 9F-1: tool_snake_jaw_fixed2_link -->
-    <link name="${prefix}tool_snake_jaw_fixed2_link">
-      <visual>
-        <origin rpy="-1.5708 0 0" xyz="0 -0.0061 0"/>
-        <geometry>
-          <mesh filename="package://dvrk_model/meshes/psm/snake_tool/gripper_1.STL"/>
+          <mesh filename="package://dvrk_model/meshes/psm/snake_tool/link_4.STL"/>
         </geometry>
       </visual>
     </link>
     <!-- Gripper  -->
-    <!-- joint 9-0: Outer open angle 1  -->
+    <!-- joint 11-0: Outer open angle 1  -->
     <joint name="jaw" type="revolute">
-      <parent link="${prefix}tool_snake_jaw_fixed2_link"/>
+      <parent link="${prefix}tool_snake_end_link"/>
       <child link="${prefix}tool_wrist_snake_ee_link_0"/>
       <axis xyz="0 0 1"/>
@@ -114,5 +80,5 @@
       <limit lower="0" upper="1.5707" velocity=".4" effort="1000"/>
     </joint>
-    <!-- link 9-0: Outer open angle virtual -->
+    <!-- link 11-0: Outer open angle virtual -->
     <link name="${prefix}tool_wrist_snake_ee_link_0">
       <visual>
@@ -123,14 +89,14 @@
       </visual>
     </link>
-    <!-- joint 9-1: Outer open angle 1  -->
+    <!-- joint 11-1: Outer open angle 1  -->
     <joint name="jaw_mimic_1" type="revolute">
-      <parent link="${prefix}tool_snake_jaw_fixed2_link"/>
+      <parent link="${prefix}tool_snake_end_link"/>
       <child link="${prefix}tool_wrist_snake_ee_link_1"/>
       <axis xyz="0 0 1"/>
-      <origin rpy="0 0.7854 0" xyz="0 -0.0061 0"/>
+      <origin rpy="0 2.3562 0" xyz="0 -0.01 0"/>
       <limit lower="-1.5707" upper="1.5707" velocity=".4" effort="1000"/>
       <mimic joint="jaw" multiplier="0.5"/>
     </joint>
-    <!-- link 9-1: Outer open angle link 1 -->
+    <!-- link 11-1: Outer open angle link 1 -->
     <link name="${prefix}tool_wrist_snake_ee_link_1">
       <visual>
@@ -141,14 +107,14 @@
       </visual>
     </link>
-    <!-- joint 9-2: Outer open angle 2   -->
+    <!-- joint 11-2: Outer open angle 2   -->
     <joint name="jaw_mimic_2" type="revolute">
-      <parent link="${prefix}tool_snake_jaw_fixed2_link"/>
+      <parent link="${prefix}tool_snake_end_link"/>
       <child link="${prefix}tool_wrist_snake_ee_link_2"/>
       <axis xyz="0 0 1"/>
-      <origin rpy="0 0.7854 0" xyz="0 -0.0061 0"/>
+      <origin rpy="0 2.3562 0" xyz="0 -0.01 0"/>
       <limit lower="-1.5707" upper="1.5707" velocity=".4" effort="1000"/>
       <mimic joint="jaw" multiplier="-0.5"/>
     </joint>
-    <!-- link 9-2: Outer open angle link 2 -->
+    <!-- link 11-2: Outer open angle link 2 -->
     <link name="${prefix}tool_wrist_snake_ee_link_2">
       <visual>
